File: EC.sch (KiCad schematic (older format))
At the start: 2 parts, among them J8 DEBUG

Commit message: Begin implementing PCI
Parts:
- removed EC1: ATSAM4E16CA-AU, IPC7351-Nominal:QFP50P1600X1600X160-100, symbol ATSAM4E16CA-AU
- added LIMB1: ATSAME70NnnA-AN, IPC7351-Nominal:QFP50P1600X1600X160-100, symbol ATSAME70NnnA-AN
Other:
- note added: "Local Integrated Management Bits - EC"
- moved on the sheet: J8
Changed lines of the file:
@@
 $EndDescr
 $Comp
-L ATSAM4E16CA-AU EC1
-U 1 1 5765D033
-P 3000 1100
-F 0 "EC1" H 3000 1267 50  0000 C CNN
-F 1 "ATSAM4E16CA-AU" H 3000 1176 50  0000 C CNN
-F 2 "IPC7351-Nominal:QFP50P1600X1600X160-100" H 3000 1500 50  0001 C CNN
-F 3 "http://www.atmel.com/Images/Atmel-11157-32-bit-Cortex-M4-Microcontroller-SAM4E16-SAM4E8_Datasheet.pdf" H 3000 1400 50  0001 C CNN
-F 4 "MCU ATMEL ATSAM4E16CA-AU" H 3000 1600 50  0001 C CNN "BOM"
-	1    3000 1100
+L CONN-10118194-0001LF-UUSB-B J8
+U 1 1 5766048A
+P 10600 1100
+F 0 "J8" H 10777 1120 50  0000 L CNN
+F 1 "DEBUG" H 10777 1029 50  0000 L CNN
+F 2 "conn-fci:CONN-10118194-0001LF-FCI" H 10600 1100 50  0001 C CNN
+F 3 "" H 10500 1300 50  0000 C CNN
+F 4 "DIST DIGIKEY 609-4618-1-ND" H 11100 2000 50  0001 C CNN "BOM"
+	1    10600 1100
 	1    0    0    -1
 $EndComp
 $Comp
-L CONN-10118194-0001LF-UUSB-B J8
-U 1 1 5766048A
-P 8000 1800
-F 0 "J8" H 8177 1820 50  0000 L CNN
-F 1 "DEBUG" H 8177 1729 50  0000 L CNN
-F 2 "conn-fci:CONN-10118194-0001LF-FCI" H 8000 1800 50  0001 C CNN
-F 3 "" H 7900 2000 50  0000 C CNN
-F 4 "DIST DIGIKEY 609-4618-1-ND" H 8500 2700 50  0001 C CNN "BOM"
-	1    8000 1800
+L ATSAME70NnnA-AN LIMB1
+U 1 1 576D1559
+P 2500 1000
+F 0 "LIMB1" H 2500 1167 50  0000 C CNN
+F 1 "ATSAME70NnnA-AN" H 2500 1076 50  0000 C CNN
+F 2 "IPC7351-Nominal:QFP50P1600X1600X160-100" H 2500 1400 50  0001 C CNN
+F 3 "http://www.atmel.com/Images/Atmel-11296-32-bit-Cortex-M7-Microcontroller-SAM-E70Q-SAM-E70N-SAM-E70J_Datasheet.pdf" H 2500 1300 50  0001 C CNN
+F 4 "MCU ATMEL ATSAME70NnnA-AN" H 2500 1500 50  0001 C CNN "BOM"
+	1    2500 1000
 	1    0    0    -1
 $EndComp
+Text Notes 600  700  0    50   ~ 0
+Local Integrated Management Bits - EC
+$Comp
+L ATSAME70NnnA-AN LIMB1
+U 2 1 576D15E6
+P 4300 1000
+F 0 "LIMB1" H 4386 1167 50  0000 C CNN
+F 1 "ATSAME70NnnA-AN" H 4386 1076 50  0000 C CNN
+F 2 "IPC7351-Nominal:QFP50P1600X1600X160-100" H 4300 1400 50  0001 C CNN
+F 3 "http://www.atmel.com/Images/Atmel-11296-32-bit-Cortex-M7-Microcontroller-SAM-E70Q-SAM-E70N-SAM-E70J_Datasheet.pdf" H 4300 1300 50  0001 C CNN
+F 4 "MCU ATMEL ATSAME70NnnA-AN" H 4300 1500 50  0001 C CNN "BOM"
+	2    4300 1000
+	1    0    0    -1
+$EndComp
+$Comp
+L ATSAME70NnnA-AN LIMB1
+U 3 1 576D162E
+P 6100 1000
+F 0 "LIMB1" H 6205 1167 50  0000 C CNN
+F 1 "ATSAME70NnnA-AN" H 6205 1076 50  0000 C CNN
+F 2 "IPC7351-Nominal:QFP50P1600X1600X160-100" H 6100 1400 50  0001 C CNN
+F 3 "http://www.atmel.com/Images/Atmel-11296-32-bit-Cortex-M7-Microcontroller-SAM-E70Q-SAM-E70N-SAM-E70J_Datasheet.pdf" H 6100 1300 50  0001 C CNN
+F 4 "MCU ATMEL ATSAME70NnnA-AN" H 6100 1500 50  0001 C CNN "BOM"
+	3    6100 1000
+	1    0    0    -1
+$EndComp
+$Comp
+L ATSAME70NnnA-AN LIMB1
+U 4 1 576D1686
+P 7900 1000
+F 0 "LIMB1" H 7980 1167 50  0000 C CNN
+F 1 "ATSAME70NnnA-AN" H 7980 1076 50  0000 C CNN
+F 2 "IPC7351-Nominal:QFP50P1600X1600X160-100" H 7900 1400 50  0001 C CNN
+F 3 "http://www.atmel.com/Images/Atmel-11296-32-bit-Cortex-M7-Microcontroller-SAM-E70Q-SAM-E70N-SAM-E70J_Datasheet.pdf" H 7900 1300 50  0001 C CNN
+F 4 "MCU ATMEL ATSAME70NnnA-AN" H 7900 1500 50  0001 C CNN "BOM"
+	4    7900 1000
+	1    0    0    -1
+$EndComp

Commit message: Uh, more misc work.
Parts:
- removed LIMB1: ATSAME70NnnA-AN, IPC7351-Nominal:QFP50P1600X1600X160-100, symbol ATSAME70NnnA-AN
- added DZ1: DRTR5V0U2SR, smd-semi:SOT-143, symbol DRTR5V0U2SR
- added LIMB1: LPC435xFET256, smd-semi:BGA100P1700X1700-256, symbol LPC435xFET256
- added Q3: 2N7002, smd-semi:SOT-23, symbol 2N7002
- added R3: 100k, IPC7351-Nominal:RESC1608X50, symbol R-0603
- added R4: 10k, IPC7351-Nominal:RESC1608X50, symbol R-0603
Connections:
- net labels added: 3V3_LIMB, GND, USB0_D+, USB0_D-, USB0_VBUS
- wire segments 0 -> 21
Other:
- note added: "WARNING: https://community.nxp.com/thread/420480"
- moved on the sheet: J8
Changed lines of the file:
@@
 $Descr A4 11693 8268
 encoding utf-8
-Sheet 7 8
+Sheet 7 9
 Title ""
 Date ""
@@
 L CONN-10118194-0001LF-UUSB-B J8
 U 1 1 5766048A
-P 10600 1100
-F 0 "J8" H 10777 1120 50  0000 L CNN
-F 1 "DEBUG" H 10777 1029 50  0000 L CNN
-F 2 "conn-fci:CONN-10118194-0001LF-FCI" H 10600 1100 50  0001 C CNN
-F 3 "" H 10500 1300 50  0000 C CNN
-F 4 "DIST DIGIKEY 609-4618-1-ND" H 11100 2000 50  0001 C CNN "BOM"
-	1    10600 1100
-	1    0    0    -1
-$EndComp
-$Comp
-L ATSAME70NnnA-AN LIMB1
-U 1 1 576D1559
-P 2500 1000
-F 0 "LIMB1" H 2500 1167 50  0000 C CNN
-F 1 "ATSAME70NnnA-AN" H 2500 1076 50  0000 C CNN
-F 2 "IPC7351-Nominal:QFP50P1600X1600X160-100" H 2500 1400 50  0001 C CNN
-F 3 "http://www.atmel.com/Images/Atmel-11296-32-bit-Cortex-M7-Microcontroller-SAM-E70Q-SAM-E70N-SAM-E70J_Datasheet.pdf" H 2500 1300 50  0001 C CNN
-F 4 "MCU ATMEL ATSAME70NnnA-AN" H 2500 1500 50  0001 C CNN "BOM"
-	1    2500 1000
-	1    0    0    -1
+P 6500 1100
+F 0 "J8" H 6677 1120 50  0000 L CNN
+F 1 "DEBUG" H 6677 1029 50  0000 L CNN
+F 2 "conn-fci:CONN-10118194-0001LF-FCI" H 6500 1100 50  0001 C CNN
+F 3 "" H 6400 1300 50  0000 C CNN
+F 4 "DIST DIGIKEY 609-4618-1-ND" H 7000 2000 50  0001 C CNN "BOM"
+	1    6500 1100
+	-1   0    0    -1
 $EndComp
 Text Notes 600  700  0    50   ~ 0
 Local Integrated Management Bits - EC
 $Comp
-L ATSAME70NnnA-AN LIMB1
-U 2 1 576D15E6
-P 4300 1000
-F 0 "LIMB1" H 4386 1167 50  0000 C CNN
-F 1 "ATSAME70NnnA-AN" H 4386 1076 50  0000 C CNN
-F 2 "IPC7351-Nominal:QFP50P1600X1600X160-100" H 4300 1400 50  0001 C CNN
-F 3 "http://www.atmel.com/Images/Atmel-11296-32-bit-Cortex-M7-Microcontroller-SAM-E70Q-SAM-E70N-SAM-E70J_Datasheet.pdf" H 4300 1300 50  0001 C CNN
-F 4 "MCU ATMEL ATSAME70NnnA-AN" H 4300 1500 50  0001 C CNN "BOM"
-	2    4300 1000
+L LPC435xFET256 LIMB1
+U 2 1 577AF03C
+P 1700 1300
+F 0 "LIMB1" H 3031 -504 50  0000 L CNN
+F 1 "LPC435xFET256" H 3031 -595 50  0000 L CNN
+F 2 "smd-semi:BGA100P1700X1700-256" H 1700 1800 50  0001 C CNN
+F 3 "http://www.nxp.com/documents/data_sheet/LPC435X_3X_2X_1X.pdf" H 1700 1700 50  0001 C CNN
+	2    1700 1300
 	1    0    0    -1
 $EndComp
 $Comp
-L ATSAME70NnnA-AN LIMB1
-U 3 1 576D162E
-P 6100 1000
-F 0 "LIMB1" H 6205 1167 50  0000 C CNN
-F 1 "ATSAME70NnnA-AN" H 6205 1076 50  0000 C CNN
-F 2 "IPC7351-Nominal:QFP50P1600X1600X160-100" H 6100 1400 50  0001 C CNN
-F 3 "http://www.atmel.com/Images/Atmel-11296-32-bit-Cortex-M7-Microcontroller-SAM-E70Q-SAM-E70N-SAM-E70J_Datasheet.pdf" H 6100 1300 50  0001 C CNN
-F 4 "MCU ATMEL ATSAME70NnnA-AN" H 6100 1500 50  0001 C CNN "BOM"
-	3    6100 1000
+L DRTR5V0U2SR DZ1
+U 1 1 577B7FBC
+P 7400 1900
+F 0 "DZ1" H 7170 1946 50  0000 R CNN
+F 1 "DRTR5V0U2SR" H 7170 1855 50  0000 R CNN
+F 2 "smd-semi:SOT-143" H 7400 1400 60  0001 C CNN
+F 3 "" H 7400 1850 60  0000 C CNN
+F 4 "TVS DIODESINC DRTR5V0U2SR" H 7400 1300 60  0001 C CNN "BOM"
+	1    7400 1900
+	-1   0    0    -1
+$EndComp
+Wire Wire Line
+	6700 900  8000 900
+Wire Wire Line
+	7400 900  7400 1500
+Wire Wire Line
+	6700 1000 7800 1000
+Wire Wire Line
+	7000 1850 7100 1850
+Wire Wire Line
+	7100 1950 6900 1950
+Wire Wire Line
+	6700 1100 7800 1100
+Wire Wire Line
+	6700 1300 6800 1300
+Wire Wire Line
+	6800 1300 6800 1500
+Wire Wire Line
+	6800 1400 6750 1400
+Connection ~ 6800 1400
+$Comp
+L GND #PWR97
+U 1 1 577B8084
+P 6800 1500
+F 0 "#PWR97" H 6800 1500 30  0001 C CNN
+F 1 "GND" H 6800 1430 30  0001 C CNN
+F 2 "" H 6800 1500 60  0000 C CNN
+F 3 "" H 6800 1500 60  0000 C CNN
+	1    6800 1500
+	-1   0    0    -1
+$EndComp
+$Comp
+L GND #PWR98
+U 1 1 577B80BD
+P 7400 2400
+F 0 "#PWR98" H 7400 2400 30  0001 C CNN
+F 1 "GND" H 7400 2330 30  0001 C CNN
+F 2 "" H 7400 2400 60  0000 C CNN
+F 3 "" H 7400 2400 60  0000 C CNN
+	1    7400 2400
+	-1   0    0    -1
+$EndComp
+Wire Wire Line
+	7400 2400 7400 2300
+Text Label 7800 1000 2    50   ~ 0
+USB0_D+
+Text Label 7800 1100 2    50   ~ 0
+USB0_D-
+Text Label 9100 1100 2    50   ~ 0
+USB0_VBUS
+Connection ~ 7400 900
+Text Label 1200 2500 0    50   ~ 0
+USB0_VBUS
+Wire Wire Line
+	1200 2500 1700 2500
+Text Label 1200 2300 0    50   ~ 0
+USB0_D+
+Wire Wire Line
+	1200 2300 1700 2300
+Text Label 1200 2400 0    50   ~ 0
+USB0_D-
+Wire Wire Line
+	1200 2400 1700 2400
+Wire Wire Line
+	6900 1950 6900 1000
+Connection ~ 6900 1000
+Wire Wire Line
+	7000 1100 7000 1850
+Connection ~ 7000 1100
+Text Notes 1300 1100 0    60   ~ 0
+WARNING: https://community.nxp.com/thread/420480
+$Comp
+L 2N7002 Q3
+U 1 1 577AFC0B
+P 8050 850
+F 0 "Q3" H 8177 896 50  0000 L CNN
+F 1 "2N7002" H 8177 805 50  0000 L CNN
+F 2 "smd-semi:SOT-23" H 8050 700 50  0001 C CNN
+F 3 "" H 8050 850 60  0000 C CNN
+F 4 "NMOS 2N7002" H 8050 600 60  0001 C CNN "BOM"
+	1    8050 850
 	1    0    0    -1
 $EndComp
+Text GLabel 7950 700  0    50   Input ~ 0
+3V3_LIMB
+Wire Wire Line
+	7950 700  8100 700
+Wire Wire Line
+	8100 700  8100 750
 $Comp
-L ATSAME70NnnA-AN LIMB1
-U 4 1 576D1686
-P 7900 1000
-F 0 "LIMB1" H 7980 1167 50  0000 C CNN
-F 1 "ATSAME70NnnA-AN" H 7980 1076 50  0000 C CNN
-F 2 "IPC7351-Nominal:QFP50P1600X1600X160-100" H 7900 1400 50  0001 C CNN
-F 3 "http://www.atmel.com/Images/Atmel-11296-32-bit-Cortex-M7-Microcontroller-SAM-E70Q-SAM-E70N-SAM-E70J_Datasheet.pdf" H 7900 1300 50  0001 C CNN
-F 4 "MCU ATMEL ATSAME70NnnA-AN" H 7900 1500 50  0001 C CNN "BOM"
-	4    7900 1000
+L R-0603 R3
+U 1 1 577B0535
+P 8100 1300
+F 0 "R3" H 8163 1346 50  0000 L CNN
+F 1 "100k" H 8163 1255 50  0000 L CNN
+F 2 "IPC7351-Nominal:RESC1608X50" H 8100 1300 50  0001 C CNN
+F 3 "" H 8100 1350 60  0000 C CNN
+F 4 "RES SMD 100k 1% [0603]" H 8850 1850 60  0001 C CNN "BOM"
+	1    8100 1300
 	1    0    0    -1
 $EndComp
+Wire Wire Line
+	8100 1200 8100 950
+$Comp
+L GND #PWR99
+U 1 1 577B0609
+P 8100 1450
+F 0 "#PWR99" H 8100 1450 30  0001 C CNN
+F 1 "GND" H 8100 1380 30  0001 C CNN
+F 2 "" H 8100 1450 60  0000 C CNN
+F 3 "" H 8100 1450 60  0000 C CNN
+	1    8100 1450
+	1    0    0    -1
+$EndComp
+Wire Wire Line
+	8100 1450 8100 1400
+$Comp
+L R-0603 R4
+U 1 1 577B0648
+P 8500 1100
+F 0 "R4" V 8608 1100 50  0000 C CNN
+F 1 "10k" V 8699 1100 50  0000 C CNN
+F 2 "IPC7351-Nominal:RESC1608X50" H 8500 1100 50  0001 C CNN
+F 3 "" H 8500 1150 60  0000 C CNN
+F 4 "RES SMD 10k 1% [0603]" H 9250 1650 60  0001 C CNN "BOM"
+	1    8500 1100
+	0    1    1    0
+$EndComp
+Wire Wire Line
+	8400 1100 8100 1100
+Connection ~ 8100 1100
+Wire Wire Line
+	9100 1100 8600 1100
 $EndSCHEMATC

Commit message: MOAR WORK
Parts:
- removed LIMB1: LPC435xFET256, smd-semi:BGA100P1700X1700-256, symbol LPC435xFET256
- added C9: 100n, IPC7351-Nominal:CAPC1005X55, symbol C-0402
- added J2: MICROSD, manuf:AMPHENOL-114-00841-68, symbol CONN-114-00841-68-MICROSD
- added LIMB1: ATSAM4S16CA-AU, IPC7351-Nominal:QFP50P1600X1600X160-100, symbol ATSAM4S16CA-AU
- added R56: 100k, IPC7351-Nominal:RESC1608X50, symbol R-0603
Connections:
- net labels added: 3V3_CARD, A0, A1, A10, A11, A12, A13, A14, A15, A16, A17, A18, A19, A2, A20, A21, A22, A23, A3, A4, A5, A6, A7, A8, A9, CARD_DET#, D0, D1, D2, D3, D4, D5, D6, D7, MCCDA, MCCK, MCDA0, MCDA1, MCDA2, MCDA3, NANDOE, NANDWE, NCS0, NCS1, NCS2, NCS3, NRD, NWAIT, NWE, SCK0, SCK1, SDA0, SDA1, USB_D+, USB_D-, USB_VBUS, XIN, XOUT
- net labels removed: USB0_D+, USB0_D-, USB0_VBUS
- wire segments 21 -> 119
Other:
- note removed: "WARNING: https://community.nxp.com/thread/420480"

Commit message: MOAR WORK, v2
Connections:
- net labels added: D[0..7], NCS
- wire segments 119 -> 107
Changed lines of the file:
@@
 $EndComp
 Wire Wire Line
-	6700 900  7400 900
-Wire Wire Line
-	7400 900  8000 900
+	6700 900  8000 900
 Wire Wire Line
 	7400 900  7400 1500
 Wire Wire Line
-	6700 1000 6900 1000
-Wire Wire Line
-	6900 1000 7800 1000
+	6700 1000 7800 1000
 Wire Wire Line
 	7000 1850 7100 1850
@@
 	7100 1950 6900 1950
 Wire Wire Line
-	6700 1100 7000 1100
-Wire Wire Line
-	7000 1100 7800 1100
+	6700 1100 7800 1100
 Wire Wire Line
 	6700 1300 6800 1300
 Wire Wire Line
-	6800 1300 6800 1400
-Wire Wire Line
-	6800 1400 6800 1500
+	6800 1300 6800 1500
 Wire Wire Line
 	6800 1400 6750 1400
@@
 $EndComp
 Wire Wire Line
-	8100 950  8100 1100
-Wire Wire Line
-	8100 1100 8100 1200
+	8100 950  8100 1200
 $Comp
 L GND #PWR101
@@
 $EndComp
 Wire Wire Line
-	10600 6300 10600 6400
-Wire Wire Line
-	10600 6400 10600 6500
-Wire Wire Line
-	10600 6500 10600 6600
-Wire Wire Line
-	10600 6600 10600 6700
-Wire Wire Line
-	10600 6700 10600 6800
+	10600 6300 10600 6800
 Wire Wire Line
 	10600 6300 10500 6300
@@
 3V3_LIMB
 Wire Wire Line
-	9100 1400 9200 1400
-Wire Wire Line
-	9200 1400 9300 1400
-Wire Wire Line
-	9200 1400 9200 1600
-Wire Wire Line
-	9200 1600 9200 1700
-Wire Wire Line
-	9200 1700 9200 1800
-Wire Wire Line
-	9200 1800 9200 1900
-Wire Wire Line
-	9200 1900 9200 2000
+	9100 1400 9300 1400
+Wire Wire Line
+	9200 1400 9200 2000
 Wire Wire Line
 	9200 1600 9300 1600
@@
 3V3_CARD
 Wire Wire Line
-	2700 2900 3400 2900
-Wire Wire Line
-	3400 2900 3800 2900
-Wire Wire Line
-	3800 2900 3900 2900
+	2700 2900 3900 2900
 $Comp
 L C-0402 C?
@@
 CARD_DET#
 Wire Wire Line
-	2800 3500 2800 3700
-Wire Wire Line
-	2800 3700 2800 3800
+	2800 3500 2800 3800
 Wire Wire Line
 	3400 3600 2700 3600
@@
 	2700 3500 2800 3500
 Connection ~ 2800 3700
+Wire Bus Line
+	6200 3600 6700 3600
+Text Label 6300 3600 0    50   ~ 0
+D[0..7]
+Text HLabel 6200 3600 0    50   BiDi ~ 0
+D[0..7]
+Text HLabel 6200 3700 0    50   Output ~ 0
+A15
+Wire Wire Line
+	6200 3700 6700 3700
+Text Label 6300 3700 0    50   ~ 0
+A15
+Text HLabel 6200 3800 0    50   Output ~ 0
+NCS
+Wire Wire Line
+	6200 3800 6700 3800
+Text Label 6300 3800 0    50   ~ 0
+NCS0
+Text HLabel 6200 3900 0    50   Output ~ 0
+NWE
+Text HLabel 6200 4000 0    50   Output ~ 0
+NRD
+Text Label 6300 3900 0    50   ~ 0
+NWE
+Text Label 6300 4000 0    50   ~ 0
+NRD
+Wire Wire Line
+	6700 3900 6200 3900
+Wire Wire Line
+	6700 4000 6200 4000
+Text Label 6300 4100 0    50   ~ 0
+NWAIT
+Text HLabel 6200 4100 0    50   Output ~ 0
+NWAIT
+Wire Wire Line
+	6700 4100 6200 4100
 $EndSCHEMATC
