File: PerBus.sch (KiCad schematic (older format))
At the start: 67 parts

Commit message: MOAR WORK, v2
Connections:
- net PCI_GNT#0: no longer PCI1.A17, PCI2.A17, PCI3.A17
- net PCI_REQ#0: no longer PCI1.B18, PCI2.B18, PCI3.B18
- new net PCI_GNT#1: PCI1.A17
- new net PCI_GNT#2: PCI2.A17
- new net PCI_GNT#3: PCI3.A17
- new net PCI_REQ#1: PCI1.B18
- new net PCI_REQ#2: PCI2.B18
- new net PCI_REQ#3: PCI3.B18
Changed lines of the file:
@@
 PCI_VIO
 Text Label 4200 2300 0    50   ~ 0
-PCI_GNT#0
+PCI_GNT#1
 $Comp
 L GND #PWR27
@@
 $EndComp
 Text Label 5700 2400 2    50   ~ 0
-PCI_REQ#0
+PCI_REQ#1
 Text Label 5700 2500 2    50   ~ 0
 PCI_VIO
@@
 PCI_VIO
 Text Label 7000 2300 0    50   ~ 0
-PCI_GNT#0
+PCI_GNT#2
 $Comp
 L GND #PWR49
@@
 $EndComp
 Text Label 8500 2400 2    50   ~ 0
-PCI_REQ#0
+PCI_REQ#2
 Text Label 8500 2500 2    50   ~ 0
 PCI_VIO
@@
 PCI_VIO
 Text Label 9800 2300 0    50   ~ 0
-PCI_GNT#0
+PCI_GNT#3
 $Comp
 L GND #PWR71
@@
 $EndComp
 Text Label 11300 2400 2    50   ~ 0
-PCI_REQ#0
+PCI_REQ#3
 Text Label 11300 2500 2    50   ~ 0
 PCI_VIO

Commit message: workworkwork
Connections:
- net PCI_AD01: no longer PCI0.B58, PCI2.B58, PCI3.B58
- net PCI_AD16: no longer PCI0.A32, PCI1.A32, PCI2.A32, PCI3.A32
- net PCI_AD17: no longer PCI0.B32, PCI1.B32, PCI2.B32, PCI3.B32
- net PCI_AD18: no longer PCI0.A31, PCI1.A31, PCI2.A31, PCI3.A31
- net PCI_AD19: no longer PCI0.B30, PCI1.B30, PCI2.B30, PCI3.B30
- net PCI_AD00 renamed AD0
- net PCI_AD02 renamed AD2
- net PCI_AD03 renamed AD3
- net PCI_AD04 renamed AD4
- net PCI_AD05 renamed AD5
- net PCI_AD06 renamed AD6
- net PCI_AD07 renamed AD7
- net PCI_AD08 renamed AD8
- net PCI_AD09 renamed AD9
- net PCI_AD10 renamed AD10
- net PCI_AD11 renamed AD11
- net PCI_AD12 renamed AD12
- net PCI_AD13 renamed AD13
- net PCI_AD14 renamed AD14
- net PCI_AD15 renamed AD15
- net PCI_AD20 renamed AD20
- net PCI_AD21 renamed AD21
- net PCI_AD22 renamed AD22
- net PCI_AD23 renamed AD23
- net PCI_AD24 renamed AD24
- net PCI_AD25 renamed AD25
- net PCI_AD26 renamed AD26
- net PCI_AD27 renamed AD27
- net PCI_AD28 renamed AD28
- net PCI_AD29 renamed AD29
- net PCI_AD30 renamed AD30
- net PCI_AD31 renamed AD31
- net PCI_CBE#0 renamed ~CBE0
- net PCI_CBE#1 renamed ~CBE1
- net PCI_CBE#2 renamed ~CBE2
- net PCI_CBE#3 renamed ~CBE3
- net PCI_CLK renamed CLK
- net PCI_DEVSEL# renamed ~DEVSEL
- net PCI_FRAME# renamed ~FRAME
- net PCI_GNT#0 renamed ~GNT0
- net PCI_GNT#1 renamed ~GNT1
- net PCI_GNT#2 renamed ~GNT2
- net PCI_GNT#3 renamed ~GNT3
- net PCI_INTA# renamed ~INT0
- net PCI_INTB# renamed ~INT1
- net PCI_INTC# renamed ~INT2
- net PCI_INTD# renamed ~INT3
- net PCI_IRDY# renamed ~IRDY
- net PCI_LOCK# renamed ~LOCK
- net PCI_M66EN renamed M66EN
- net PCI_PAR renamed PAR
- net PCI_PERR# renamed ~PERR
- net PCI_PME# renamed ~PME
- net PCI_PRSNT1#0 renamed ~PRSNT1_0
- net PCI_PRSNT1#1 renamed ~PRSNT1_1
- net PCI_PRSNT1#2 renamed ~PRSNT1_2
- net PCI_PRSNT1#3 renamed ~PRSNT1_3
- net PCI_PRSNT2#0 renamed ~PRSNT2_0
- net PCI_PRSNT2#1 renamed ~PRSNT2_1
- net PCI_PRSNT2#2 renamed ~PRSNT2_2
- net PCI_PRSNT2#3 renamed ~PRSNT2_3
- net PCI_REQ#0 renamed ~REQ0
- net PCI_REQ#1 renamed ~REQ1
- net PCI_REQ#2 renamed ~REQ2
- net PCI_REQ#3 renamed ~REQ3
- net PCI_RST# renamed ~RST
- net PCI_SERR# renamed ~SERR
- net PCI_SMBCLK renamed SCL
- net PCI_SMBDAT renamed SDA
- net PCI_STOP# renamed ~STOP
- net PCI_TRDY# renamed ~TRDY
- new net AD1: PCI0.B58, PCI2.B58, PCI3.B58
- new net AD16: PCI0.A32, PCI1.A32, PCI2.A32, PCI3.A32
- new net AD17: PCI0.B32, PCI1.B32, PCI2.B32, PCI3.B32
- new net AD18: PCI0.A31, PCI1.A31, PCI2.A31, PCI3.A31
- new net AD19: PCI0.B30, PCI1.B30, PCI2.B30, PCI3.B30
Other:
- note removed: "5V: 25W 5A\n3.3V: 25W 7.6A\n12V: 6W 500mA\n-12V: 1.2W 100mA\n3v3aux: 1.3W 375mA\nVio: 5W 1.5A"
- moved on the sheet: C67, C68, C69, C70, R49
