File: Blinkenlights.sch (KiCad schematic (older format))
At the start: 91 parts, among them J1 PDI, U1 ATXMEGA8E5-MU

Commit message: Route CPU bus and cache
Parts:
- removed DS19: BRG_P2V5(R), smd-semi:LED-0603, symbol LED-0603
- removed DS20: CPU_P2V5(R), smd-semi:LED-0603, symbol LED-0603
- removed DS21: BRG_P2V5(G), smd-semi:LED-0603, symbol LED-0603
- removed DS22: CPU_P2V5(G), smd-semi:LED-0603, symbol LED-0603
Changed lines of the file:
@@
-$EndComp
-$Comp
-L LED-0603 DS19
-U 1 1 577C48ED
-P 8500 2300
-F 0 "DS19" H 8650 2346 50  0000 L CNN
-F 1 "BRG_P2V5(R)" H 8650 2255 50  0000 L CNN
-F 2 "smd-semi:LED-0603" H 8500 2150 50  0001 C CNN
-F 3 "" H 8500 2300 60  0000 C CNN
-F 4 "LED RED [0603]" H 8500 2050 60  0001 C CNN "BOM"
-	1    8500 2300
-	1    0    0    -1
-$EndComp
-$Comp
-L LED-0603 DS21
-U 1 1 577C48F4
-P 9300 2300
-F 0 "DS21" H 9450 2346 50  0000 L CNN
-F 1 "BRG_P2V5(G)" H 9450 2255 50  0000 L CNN
-F 2 "smd-semi:LED-0603" H 9300 2150 50  0001 C CNN
-F 3 "" H 9300 2300 60  0000 C CNN
-F 4 "LED GREEN [0603]" H 9300 2050 60  0001 C CNN "BOM"
-	1    9300 2300
-	1    0    0    -1
 $EndComp
 $Comp
@@
 F 4 "LED GREEN [0603]" H 7400 3450 60  0001 C CNN "BOM"
 	1    7400 3700
-	1    0    0    -1
-$EndComp
-$Comp
-L LED-0603 DS20
-U 1 1 577C746A
-P 8500 3700
-F 0 "DS20" H 8650 3746 50  0000 L CNN
-F 1 "CPU_P2V5(R)" H 8650 3655 50  0000 L CNN
-F 2 "smd-semi:LED-0603" H 8500 3550 50  0001 C CNN
-F 3 "" H 8500 3700 60  0000 C CNN
-F 4 "LED RED [0603]" H 8500 3450 60  0001 C CNN "BOM"
-	1    8500 3700
-	1    0    0    -1
-$EndComp
-$Comp
-L LED-0603 DS22
-U 1 1 577C7471
-P 9300 3700
-F 0 "DS22" H 9450 3746 50  0000 L CNN
-F 1 "CPU_P2V5(G)" H 9450 3655 50  0000 L CNN
-F 2 "smd-semi:LED-0603" H 9300 3550 50  0001 C CNN
-F 3 "" H 9300 3700 60  0000 C CNN
-F 4 "LED GREEN [0603]" H 9300 3450 60  0001 C CNN "BOM"
-	1    9300 3700
 	1    0    0    -1
 $EndComp
@@
 SCL
 $Comp
-L GND #PWR128
+L GND #PWR138
 U 1 1 577CE6F2
 P 2300 9500
-F 0 "#PWR128" H 2300 9500 30  0001 C CNN
+F 0 "#PWR138" H 2300 9500 30  0001 C CNN
 F 1 "GND" H 2300 9430 30  0001 C CNN
 F 2 "" H 2300 9500 60  0000 C CNN
@@
 Connection ~ 1400 6500
 $Comp
-L GND #PWR125
+L GND #PWR135
 U 1 1 577B3D62
 P 1400 7750
-F 0 "#PWR125" H 1400 7750 30  0001 C CNN
+F 0 "#PWR135" H 1400 7750 30  0001 C CNN
 F 1 "GND" H 1400 7680 30  0001 C CNN
 F 2 "" H 1400 7750 60  0000 C CNN
@@
 Connection ~ 1950 6500
 $Comp
-L GND #PWR127
+L GND #PWR137
 U 1 1 577B9706
 P 1950 6800
-F 0 "#PWR127" H 1950 6800 30  0001 C CNN
+F 0 "#PWR137" H 1950 6800 30  0001 C CNN
 F 1 "GND" H 1950 6730 30  0001 C CNN
 F 2 "" H 1950 6800 60  0000 C CNN
@@
 	1950 6800 1950 6750
 $Comp
-L GND #PWR126
+L GND #PWR136
 U 1 1 577B9A2E
 P 1550 6800
-F 0 "#PWR126" H 1550 6800 30  0001 C CNN
+F 0 "#PWR136" H 1550 6800 30  0001 C CNN
 F 1 "GND" H 1550 6730 30  0001 C CNN
 F 2 "" H 1550 6800 60  0000 C CNN

Commit message: workworkwork
Parts:
- removed R14, R17, R22, R52, R55, R8, R9: 51k, IPC7351-Nominal:RESC1608X50, symbol R-0603
Connections:
- net SBY_P3V3 renamed P3V3_STBY
Other:
- note removed: "Set I2C address by population of pullups\nPresent = 1, absent = 0"
Changed lines of the file:
@@
 $Descr B 17000 11000
 encoding utf-8
-Sheet 8 9
+Sheet 8 10
 Title ""
 Date ""
@@
 SCL
 $Comp
-L GND #PWR138
+L GND #PWR144
 U 1 1 577CE6F2
 P 2300 9500
-F 0 "#PWR138" H 2300 9500 30  0001 C CNN
+F 0 "#PWR144" H 2300 9500 30  0001 C CNN
 F 1 "GND" H 2300 9430 30  0001 C CNN
 F 2 "" H 2300 9500 60  0000 C CNN
@@
 	1    0    0    -1
 $EndComp
-$Comp
-L R-0603 R8
-U 1 1 577D1AE1
-P 4400 6700
-F 0 "R8" H 4463 6746 50  0000 L CNN
-F 1 "51k" H 4463 6655 50  0000 L CNN
-F 2 "IPC7351-Nominal:RESC1608X50" H 4400 6700 50  0001 C CNN
-F 3 "" H 4400 6750 60  0000 C CNN
-F 4 "RES SMD 51k 1% [0603]" H 5150 7250 60  0001 C CNN "BOM"
-	1    4400 6700
-	1    0    0    -1
-$EndComp
-$Comp
-L R-0603 R9
-U 1 1 577D1D2F
-P 4700 6700
-F 0 "R9" H 4763 6746 50  0000 L CNN
-F 1 "51k" H 4763 6655 50  0000 L CNN
-F 2 "IPC7351-Nominal:RESC1608X50" H 4700 6700 50  0001 C CNN
-F 3 "" H 4700 6750 60  0000 C CNN
-F 4 "RES SMD 51k 1% [0603]" H 5450 7250 60  0001 C CNN "BOM"
-	1    4700 6700
-	1    0    0    -1
-$EndComp
-$Comp
-L R-0603 R14
-U 1 1 577D1E0F
-P 5000 6700
-F 0 "R14" H 5063 6746 50  0000 L CNN
-F 1 "51k" H 5063 6655 50  0000 L CNN
-F 2 "IPC7351-Nominal:RESC1608X50" H 5000 6700 50  0001 C CNN
-F 3 "" H 5000 6750 60  0000 C CNN
-F 4 "RES SMD 51k 1% [0603]" H 5750 7250 60  0001 C CNN "BOM"
-	1    5000 6700
-	1    0    0    -1
-$EndComp
-$Comp
-L R-0603 R17
-U 1 1 577D1EF2
-P 5300 6700
-F 0 "R17" H 5363 6746 50  0000 L CNN
-F 1 "51k" H 5363 6655 50  0000 L CNN
-F 2 "IPC7351-Nominal:RESC1608X50" H 5300 6700 50  0001 C CNN
-F 3 "" H 5300 6750 60  0000 C CNN
-F 4 "RES SMD 51k 1% [0603]" H 6050 7250 60  0001 C CNN "BOM"
-	1    5300 6700
-	1    0    0    -1
-$EndComp
-$Comp
-L R-0603 R22
-U 1 1 577D1FD8
-P 5600 6700
-F 0 "R22" H 5663 6746 50  0000 L CNN
-F 1 "51k" H 5663 6655 50  0000 L CNN
-F 2 "IPC7351-Nominal:RESC1608X50" H 5600 6700 50  0001 C CNN
-F 3 "" H 5600 6750 60  0000 C CNN
-F 4 "RES SMD 51k 1% [0603]" H 6350 7250 60  0001 C CNN "BOM"
-	1    5600 6700
-	1    0    0    -1
-$EndComp
-$Comp
-L R-0603 R52
-U 1 1 577D20C1
-P 5900 6700
-F 0 "R52" H 5963 6746 50  0000 L CNN
-F 1 "51k" H 5963 6655 50  0000 L CNN
-F 2 "IPC7351-Nominal:RESC1608X50" H 5900 6700 50  0001 C CNN
-F 3 "" H 5900 6750 60  0000 C CNN
-F 4 "RES SMD 51k 1% [0603]" H 6650 7250 60  0001 C CNN "BOM"
-	1    5900 6700
-	1    0    0    -1
-$EndComp
-$Comp
-L R-0603 R55
-U 1 1 577D21AD
-P 6200 6700
-F 0 "R55" H 6263 6746 50  0000 L CNN
-F 1 "51k" H 6263 6655 50  0000 L CNN
-F 2 "IPC7351-Nominal:RESC1608X50" H 6200 6700 50  0001 C CNN
-F 3 "" H 6200 6750 60  0000 C CNN
-F 4 "RES SMD 51k 1% [0603]" H 6950 7250 60  0001 C CNN "BOM"
-	1    6200 6700
-	1    0    0    -1
-$EndComp
 Text GLabel 1300 6500 0    50   Input ~ 0
-SBY_P3V3
+P3V3_STBY
 $Comp
 L R-0603 R10
@@
 	0    1    1    0
 $EndComp
-Text Notes 4400 6450 0    50   ~ 0
-Set I2C address by population of pullups\nPresent = 1, absent = 0
 $Comp
 L CONN-100MIL-M-2x3 J1
@@
 Wire Wire Line
 	2300 7000 2400 7000
-Connection ~ 2300 6500
 Wire Wire Line
 	2300 6500 2300 7150
 Wire Wire Line
 	2400 6900 2300 6900
-Connection ~ 4400 6500
-Connection ~ 4700 6500
-Wire Wire Line
-	4700 6500 4700 6600
-Connection ~ 5000 6500
-Wire Wire Line
-	5000 6500 5000 6600
-Connection ~ 5300 6500
-Wire Wire Line
-	5300 6500 5300 6600
-Connection ~ 5600 6500
-Wire Wire Line
-	5600 6500 5600 6600
-Connection ~ 5900 6500
-Wire Wire Line
-	5900 6500 5900 6600
-Wire Wire Line
-	6200 6500 6200 6600
-Wire Wire Line
-	1300 6500 6200 6500
-Wire Wire Line
-	4400 6500 4400 6600
-Connection ~ 6200 7500
-Wire Wire Line
-	6200 6800 6200 7500
-Connection ~ 5900 7400
-Wire Wire Line
-	5900 6800 5900 7400
-Connection ~ 5600 7300
-Wire Wire Line
-	5600 6800 5600 7300
-Connection ~ 5300 7200
-Wire Wire Line
-	5300 6800 5300 7200
-Connection ~ 5000 7100
-Wire Wire Line
-	5000 6800 5000 7100
-Connection ~ 4700 7000
-Wire Wire Line
-	4700 6800 4700 7000
-Connection ~ 4400 6900
-Wire Wire Line
-	4400 6800 4400 6900
 Connection ~ 2300 9400
 Wire Wire Line
@@
 Wire Wire Line
 	4300 7800 4200 7800
-Wire Wire Line
-	6800 7600 4200 7600
-Wire Wire Line
-	4200 7500 6800 7500
-Wire Wire Line
-	4200 7400 6800 7400
-Wire Wire Line
-	4200 7300 6800 7300
-Wire Wire Line
-	4200 7200 6800 7200
-Wire Wire Line
-	4200 7100 6800 7100
-Wire Wire Line
-	4200 7000 6800 7000
-Wire Wire Line
-	4200 6900 6800 6900
 Wire Wire Line
 	9300 3550 9300 3600
@@
 Connection ~ 1400 6500
 $Comp
-L GND #PWR135
+L GND #PWR141
 U 1 1 577B3D62
 P 1400 7750
-F 0 "#PWR135" H 1400 7750 30  0001 C CNN
+F 0 "#PWR141" H 1400 7750 30  0001 C CNN
 F 1 "GND" H 1400 7680 30  0001 C CNN
 F 2 "" H 1400 7750 60  0000 C CNN
@@
 Connection ~ 1950 6500
 $Comp
-L GND #PWR137
+L GND #PWR143
 U 1 1 577B9706
 P 1950 6800
-F 0 "#PWR137" H 1950 6800 30  0001 C CNN
+F 0 "#PWR143" H 1950 6800 30  0001 C CNN
 F 1 "GND" H 1950 6730 30  0001 C CNN
 F 2 "" H 1950 6800 60  0000 C CNN
@@
 	1950 6800 1950 6750
 $Comp
-L GND #PWR136
+L GND #PWR142
 U 1 1 577B9A2E
 P 1550 6800
-F 0 "#PWR136" H 1550 6800 30  0001 C CNN
+F 0 "#PWR142" H 1550 6800 30  0001 C CNN
 F 1 "GND" H 1550 6730 30  0001 C CNN
 F 2 "" H 1550 6800 60  0000 C CNN
@@
 Wire Wire Line
 	1550 6800 1550 6750
+Wire Wire Line
+	2300 6500 1300 6500
+Wire Wire Line
+	6800 6900 4200 6900
+Wire Wire Line
+	6800 7000 4200 7000
+Wire Wire Line
+	6800 7100 4200 7100
+Wire Wire Line
+	6800 7200 4200 7200
+Wire Wire Line
+	6800 7300 4200 7300
+Wire Wire Line
+	6800 7400 4200 7400
+Wire Wire Line
+	6800 7500 4200 7500
+Wire Wire Line
+	6800 7600 4200 7600
 $EndSCHEMATC
