File: CPUn.sch (KiCad schematic (older format))
At the start: 1 part

Commit message: Uh, more misc work.
Parts:
- removed CPU0: XC6SLX16-2FTG256C, manuf:XILINX-FT256, symbol XC6SLX16-2FTG256C
- added CPU0: XC6SLX25-FGG484, manuf:XILINX-FGG484, symbol XC6SLX25-FGG484
Changed lines of the file:
@@
 $Descr A4 11693 8268
 encoding utf-8
-Sheet 5 8
+Sheet 5 9
 Title ""
 Date ""
@@
 $EndDescr
 $Comp
-L XC6SLX16-2FTG256C CPU0
-U 1 1 5765A948
-P 3000 1500
-AR Path="/5765A5BA/5765A948" Ref="CPU0"  Part="1"
-AR Path="/5765B2E6/5765A948" Ref="CPU1"  Part="1"
-F 0 "CPU1" H 4069 -360 50  0000 L CNN
-F 1 "XC6SLX16-2FTG256C" H 4069 -451 50  0000 L CNN
-F 2 "manuf:XILINX-FT256" H 3000 1500 50  0001 C CNN
-F 3 "" H 1400 1600 50  0000 C CNN
-F 4 "IC XILINX XC6SLX16-2FTG256C" H 4100 2250 60  0001 C CNN "BOM"
-	1    3000 1500
+L XC6SLX25-FGG484 CPU0
+U 1 1 577B458D
+P 5200 1400
+AR Path="/5765A5BA/577B458D" Ref="CPU0"  Part="1"
+AR Path="/5765B2E6/577B458D" Ref="CPU1"  Part="1"
+F 0 "CPU1" H 6331 -1904 50  0000 L CNN
+F 1 "XC6SLX25-FGG484" H 6331 -1995 50  0000 L CNN
+F 2 "manuf:XILINX-FGG484" H 5300 1550 50  0001 C CNN
+F 3 "" H 5400 1650 60  0001 C CNN
+	1    5200 1400
 	1    0    0    -1
 $EndComp

Commit message: workworkwork
Parts:
- added U2: AS7C38098A, IPC7351-Nominal:SOP80P1176X120-44, symbol AS7C38098A
Connections:
- net labels added: ADDR#, BUSACK#, BUSCLK, BUSINT#, BUSREQ#, D[0..31], P3V3_CPU, WAIT#, WR#
- wire segments 0 -> 12
Other:
- note added: "CACHE RAM: AS7C38098A-10TIN"
- moved on the sheet: CPU1A
Changed lines of the file:
@@
 LIBS:Xilinx
 LIBS:Richtek
+LIBS:semi-diode-Panasonic
 LIBS:c4puter-cache
 EELAYER 25 0
 EELAYER END
-$Descr A4 11693 8268
+$Descr B 17000 11000
 encoding utf-8
-Sheet 5 9
+Sheet 4 10
 Title ""
 Date ""
@@
 L XC6SLX25-FGG484 CPU0
 U 1 1 577B458D
-P 5200 1400
-AR Path="/5765A5BA/577B458D" Ref="CPU0"  Part="1"
+P 3800 700
+AR Path="/5765A5BA/577B458D" Ref="CPU0"  Part="3"
 AR Path="/5765B2E6/577B458D" Ref="CPU1"  Part="1"
-F 0 "CPU1" H 6331 -1904 50  0000 L CNN
-F 1 "XC6SLX25-FGG484" H 6331 -1995 50  0000 L CNN
-F 2 "manuf:XILINX-FGG484" H 5300 1550 50  0001 C CNN
-F 3 "" H 5400 1650 60  0001 C CNN
-	1    5200 1400
+F 0 "CPU1" H 4931 -2604 50  0000 L CNN
+F 1 "XC6SLX25-FGG484" H 4931 -2695 50  0000 L CNN
+F 2 "manuf:XILINX-FGG484" H 3900 850 50  0001 C CNN
+F 3 "" H 4000 950 60  0001 C CNN
+	1    3800 700
 	1    0    0    -1
 $EndComp
+Text HLabel 2000 1800 0    50   BiDi ~ 0
+D[0..31]
+Text HLabel 2000 1900 0    50   Input ~ 0
+WAIT#
+Text HLabel 2000 2000 0    50   Output ~ 0
+ADDR#
+Text HLabel 2000 2100 0    50   Output ~ 0
+WR#
+Text HLabel 2000 2200 0    50   Output ~ 0
+BUSCLK
+Text HLabel 2000 2300 0    50   Output ~ 0
+BUSREQ#
+Text HLabel 2000 2400 0    50   Input ~ 0
+BUSACK#
+Text HLabel 2000 2500 0    50   Input ~ 0
+BUSINT#
+Text Notes 1000 800  0    50   ~ 0
+CACHE RAM: AS7C38098A-10TIN
+Text GLabel 3600 9000 0    50   Input ~ 0
+P3V3_CPU
+Wire Wire Line
+	3600 9000 3800 9000
+Wire Wire Line
+	3700 9100 3800 9100
+Connection ~ 3700 9000
+Connection ~ 3700 9100
+Connection ~ 3700 9200
+Connection ~ 3700 9300
+Connection ~ 3700 9400
+Connection ~ 3700 9500
+Connection ~ 3700 9600
+Connection ~ 3700 9700
+Connection ~ 3700 9800
+Connection ~ 3700 9900
+Wire Wire Line
+	3700 9200 3800 9200
+Wire Wire Line
+	3700 9300 3800 9300
+Wire Wire Line
+	3700 9400 3800 9400
+Wire Wire Line
+	3700 9500 3800 9500
+Wire Wire Line
+	3700 9600 3800 9600
+Wire Wire Line
+	3700 9700 3800 9700
+Wire Wire Line
+	3700 9800 3800 9800
+Wire Wire Line
+	3700 9900 3800 9900
+Wire Wire Line
+	3700 10000 3800 10000
+Wire Wire Line
+	3700 9000 3700 10000
+$Comp
+L AS7C38098A U2
+U 1 1 5783D342
+P 15000 4200
+AR Path="/5765A5BA/5783D342" Ref="U2"  Part="1"
+AR Path="/5765B2E6/5783D342" Ref="U3"  Part="1"
+F 0 "U3" H 15000 4467 50  0000 C CNN
+F 1 "AS7C38098A" H 15000 4376 50  0000 C CNN
+F 2 "IPC7351-Nominal:SOP80P1176X120-44" H 15000 1700 50  0001 C CNN
+F 3 "http://www.alliancememory.com/pdf/sram/fa/as7c38098a.pdf" H 15000 1600 50  0001 C CNN
+F 4 "DIST DIGIKEY 1450-1069-ND" H 15000 4200 60  0001 C CNN "BOM"
+	1    15000 4200
+	1    0    0    -1
+$EndComp

Commit message: Route CPU bus and cache
Parts:
- added C75, C76: 1u, IPC7351-Nominal:CAPC1005X55, symbol C-0402
- added unit 4 of CPU0
- added unit 1 of CPU0
- added unit 2 of CPU0
- renumbered U2 to CACHE0
Connections:
- net labels added: CACHE_A0, CACHE_A1, CACHE_A10, CACHE_A11, CACHE_A12, CACHE_A13, CACHE_A14, CACHE_A15, CACHE_A16, CACHE_A17, CACHE_A18, CACHE_A2, CACHE_A3, CACHE_A4, CACHE_A5, CACHE_A6, CACHE_A7, CACHE_A8, CACHE_A9, CACHE_DQ0, CACHE_DQ1, CACHE_DQ10, CACHE_DQ11, CACHE_DQ12, CACHE_DQ13, CACHE_DQ14, CACHE_DQ15, CACHE_DQ2, CACHE_DQ3, CACHE_DQ4, CACHE_DQ5, CACHE_DQ6, CACHE_DQ7, CACHE_DQ8, CACHE_DQ9, CACHE_~CE, CACHE_~LB, CACHE_~OE, CACHE_~UB, CACHE_~WE, CPUID0, CPUID1, D0, D1, D10, D11, D12, D13, D14, D15, D16, D17, D18, D19, D2, D20, D21, D22, D23, D24, D25, D26, D27, D28, D29, D3, D30, D31, D4, D5, D6, D7, D8, D9, GND, P1V5_BRIDGE
- wire segments 12 -> 168
Other:
- moved on the sheet: CACHE0

Commit message: workworkwork
Changed lines of the file:
@@
 $Descr C 22000 17000
 encoding utf-8
-Sheet 5 9
+Sheet 4 10
 Title ""
 Date ""
@@
 AR Path="/5765A5BA/577B458D" Ref="CPU0"  Part="3"
 AR Path="/5765B2E6/577B458D" Ref="CPU1"  Part="3"
-F 0 "CPU0" H 5431 -3904 50  0000 L CNN
+F 0 "CPU1" H 5431 -3904 50  0000 L CNN
 F 1 "XC6SLX25-FGG484" H 5431 -3995 50  0000 L CNN
 F 2 "manuf:XILINX-FGG484" H 3900 850 50  0001 C CNN
@@
 AR Path="/5765A5BA/5783D342" Ref="CACHE0"  Part="1"
 AR Path="/5765B2E6/5783D342" Ref="CACHE1"  Part="1"
-F 0 "CACHE0" H 19500 7467 50  0000 C CNN
+F 0 "CACHE1" H 19500 7467 50  0000 C CNN
 F 1 "AS7C38098A" H 19500 7376 50  0000 C CNN
 F 2 "IPC7351-Nominal:SOP80P1176X120-44" H 19500 4700 50  0001 C CNN
@@
 AR Path="/5765A5BA/5793B4AE" Ref="#PWR111"  Part="1"
 AR Path="/5765B2E6/5793B4AE" Ref="#PWR113"  Part="1"
-F 0 "#PWR111" H 20200 9600 30  0001 C CNN
+F 0 "#PWR113" H 20200 9600 30  0001 C CNN
 F 1 "GND" H 20200 9530 30  0001 C CNN
 F 2 "" H 20200 9600 60  0000 C CNN
@@
 AR Path="/5765A5BA/5793BAAD" Ref="C75"  Part="1"
 AR Path="/5765B2E6/5793BAAD" Ref="C77"  Part="1"
-F 0 "C75" H 20313 10046 50  0000 L CNN
+F 0 "C77" H 20313 10046 50  0000 L CNN
 F 1 "1u" H 20313 9955 50  0000 L CNN
 F 2 "IPC7351-Nominal:CAPC1005X55" H 20200 10000 50  0001 C CNN
@@
 AR Path="/5765A5BA/5793BB4A" Ref="C76"  Part="1"
 AR Path="/5765B2E6/5793BB4A" Ref="C78"  Part="1"
-F 0 "C76" H 20713 10046 50  0000 L CNN
+F 0 "C78" H 20713 10046 50  0000 L CNN
 F 1 "1u" H 20713 9955 50  0000 L CNN
 F 2 "IPC7351-Nominal:CAPC1005X55" H 20600 10000 50  0001 C CNN
@@
 AR Path="/5765A5BA/5793BC86" Ref="#PWR112"  Part="1"
 AR Path="/5765B2E6/5793BC86" Ref="#PWR114"  Part="1"
-F 0 "#PWR112" H 20400 10300 30  0001 C CNN
+F 0 "#PWR114" H 20400 10300 30  0001 C CNN
 F 1 "GND" H 20400 10230 30  0001 C CNN
 F 2 "" H 20400 10300 60  0000 C CNN
@@
 AR Path="/5765A5BA/57942A58" Ref="CPU0"  Part="4"
 AR Path="/5765B2E6/57942A58" Ref="CPU1"  Part="4"
-F 0 "CPU0" H 9031 -2854 50  0000 L CNN
+F 0 "CPU1" H 9031 -2854 50  0000 L CNN
 F 1 "XC6SLX25-FGG484" H 9031 -2945 50  0000 L CNN
 F 2 "manuf:XILINX-FGG484" H 7300 950 50  0001 C CNN
@@
 AR Path="/5765A5BA/5795C53B" Ref="CPU0"  Part="1"
 AR Path="/5765B2E6/5795C53B" Ref="CPU1"  Part="1"
-F 0 "CPU0" H 12131 -2104 50  0000 L CNN
+F 0 "CPU1" H 12131 -2104 50  0000 L CNN
 F 1 "XC6SLX25-FGG484" H 12131 -2195 50  0000 L CNN
 F 2 "manuf:XILINX-FGG484" H 11100 1350 50  0001 C CNN
@@
 AR Path="/5765A5BA/5795C751" Ref="CPU0"  Part="2"
 AR Path="/5765B2E6/5795C751" Ref="CPU1"  Part="2"
-F 0 "CPU0" H 15331 -2304 50  0000 L CNN
+F 0 "CPU1" H 15331 -2304 50  0000 L CNN
 F 1 "XC6SLX25-FGG484" H 15331 -2395 50  0000 L CNN
 F 2 "manuf:XILINX-FGG484" H 13700 1450 50  0001 C CNN

Commit message: TODO: learn to write good commit messages
Connections:
- net PROGRAM_B: now reaches CPU0.AA1 (PROGRAM_B_2)
- net DIN: now reaches CPU0.AA20 (IO_L3P_D0_DIN_MISO_MISO1_2)
- net INIT_B: now reaches CPU0.T6 (IO_L65P_INIT_B_2)
- net CCLK: now reaches CPU0.Y21 (IO_L1P_CCLK_2)
- net DONE: now reaches CPU0.Y22 (DONE_2)
- no-connect marks 0 -> 2
Changed lines of the file:
@@
 LIBS:semi-diode-Panasonic
 LIBS:Murata
+LIBS:semi-trans-Panasonic
 LIBS:c4puter-cache
 EELAYER 25 0
@@
 AR Path="/5765A5BA/577B458D" Ref="CPU0"  Part="3"
 AR Path="/5765B2E6/577B458D" Ref="CPU1"  Part="3"
-F 0 "CPU1" H 5431 -3904 50  0000 L CNN
+F 0 "CPU0" H 5431 -3904 50  0000 L CNN
 F 1 "XC6SLX25-FGG484" H 5431 -3995 50  0000 L CNN
 F 2 "manuf:XILINX-FGG484" H 3900 850 50  0001 C CNN
@@
 AR Path="/5765A5BA/5783D342" Ref="CACHE0"  Part="1"
 AR Path="/5765B2E6/5783D342" Ref="CACHE1"  Part="1"
-F 0 "CACHE1" H 19500 7467 50  0000 C CNN
+F 0 "CACHE0" H 19500 7467 50  0000 C CNN
 F 1 "AS7C38098A" H 19500 7376 50  0000 C CNN
 F 2 "IPC7351-Nominal:SOP80P1176X120-44" H 19500 4700 50  0001 C CNN
@@
 P3V3_CPU
 $Comp
-L GND #PWR112
+L GND #PWR119
 U 1 1 5793B4AE
 P 20200 9600
-AR Path="/5765A5BA/5793B4AE" Ref="#PWR112"  Part="1"
-AR Path="/5765B2E6/5793B4AE" Ref="#PWR114"  Part="1"
-F 0 "#PWR114" H 20200 9600 30  0001 C CNN
+AR Path="/5765A5BA/5793B4AE" Ref="#PWR119"  Part="1"
+AR Path="/5765B2E6/5793B4AE" Ref="#PWR121"  Part="1"
+F 0 "#PWR119" H 20200 9600 30  0001 C CNN
 F 1 "GND" H 20200 9530 30  0001 C CNN
 F 2 "" H 20200 9600 60  0000 C CNN
@@
 AR Path="/5765A5BA/5793BAAD" Ref="C75"  Part="1"
 AR Path="/5765B2E6/5793BAAD" Ref="C77"  Part="1"
-F 0 "C77" H 20313 10046 50  0000 L CNN
+F 0 "C75" H 20313 10046 50  0000 L CNN
 F 1 "1u" H 20313 9955 50  0000 L CNN
 F 2 "IPC7351-Nominal:CAPC1005X55" H 20200 10000 50  0001 C CNN
@@
 AR Path="/5765A5BA/5793BB4A" Ref="C76"  Part="1"
 AR Path="/5765B2E6/5793BB4A" Ref="C78"  Part="1"
-F 0 "C78" H 20713 10046 50  0000 L CNN
+F 0 "C76" H 20713 10046 50  0000 L CNN
 F 1 "1u" H 20713 9955 50  0000 L CNN
 F 2 "IPC7351-Nominal:CAPC1005X55" H 20600 10000 50  0001 C CNN
@@
 $EndComp
 $Comp
-L GND #PWR113
+L GND #PWR120
 U 1 1 5793BC86
 P 20400 10300
-AR Path="/5765A5BA/5793BC86" Ref="#PWR113"  Part="1"
-AR Path="/5765B2E6/5793BC86" Ref="#PWR115"  Part="1"
-F 0 "#PWR115" H 20400 10300 30  0001 C CNN
+AR Path="/5765A5BA/5793BC86" Ref="#PWR120"  Part="1"
+AR Path="/5765B2E6/5793BC86" Ref="#PWR122"  Part="1"
+F 0 "#PWR120" H 20400 10300 30  0001 C CNN
 F 1 "GND" H 20400 10230 30  0001 C CNN
 F 2 "" H 20400 10300 60  0000 C CNN
@@
 AR Path="/5765A5BA/57942A58" Ref="CPU0"  Part="4"
 AR Path="/5765B2E6/57942A58" Ref="CPU1"  Part="4"
-F 0 "CPU1" H 9031 -2854 50  0000 L CNN
+F 0 "CPU0" H 9031 -2854 50  0000 L CNN
 F 1 "XC6SLX25-FGG484" H 9031 -2945 50  0000 L CNN
 F 2 "manuf:XILINX-FGG484" H 7300 950 50  0001 C CNN
@@
 Connection ~ 7100 8100
 Wire Wire Line
-	7100 8200 7100 7200
+	7100 7200 7100 8200
 Wire Wire Line
 	6900 800  7200 800
@@
 AR Path="/5765A5BA/5795C53B" Ref="CPU0"  Part="1"
 AR Path="/5765B2E6/5795C53B" Ref="CPU1"  Part="1"
-F 0 "CPU1" H 12131 -2104 50  0000 L CNN
+F 0 "CPU0" H 12131 -2104 50  0000 L CNN
 F 1 "XC6SLX25-FGG484" H 12131 -2195 50  0000 L CNN
 F 2 "manuf:XILINX-FGG484" H 11100 1350 50  0001 C CNN
@@
 AR Path="/5765A5BA/5795C751" Ref="CPU0"  Part="2"
 AR Path="/5765B2E6/5795C751" Ref="CPU1"  Part="2"
-F 0 "CPU1" H 15331 -2304 50  0000 L CNN
+F 0 "CPU0" H 15331 -2304 50  0000 L CNN
 F 1 "XC6SLX25-FGG484" H 15331 -2395 50  0000 L CNN
 F 2 "manuf:XILINX-FGG484" H 13700 1450 50  0001 C CNN
@@
 Wire Wire Line
 	13100 3800 13600 3800
+Text HLabel 3600 1300 0    50   Input ~ 0
+DIN
+Text HLabel 3600 900  0    50   Input ~ 0
+CCLK
+Text HLabel 3700 8900 0    50   Input ~ 0
+PROGRAM_B
+Text HLabel 3600 800  0    50   Output ~ 0
+DONE
+Text HLabel 3700 8700 0    50   Output ~ 0
+INIT_B
+Wire Wire Line
+	3600 900  3800 900
+Wire Wire Line
+	3600 800  3800 800
+Wire Wire Line
+	3600 1300 3800 1300
+NoConn ~ 3800 1400
+Wire Wire Line
+	3700 8700 3800 8700
+NoConn ~ 3800 8800
+Wire Wire Line
+	3700 8900 3800 8900
 $EndSCHEMATC
