File: Misc.sch (KiCad schematic (older format))
At the start: 14 parts, among them U3 PCF8523TK, U4 TLV70218DBV, U5 CDCE913PW, X1 32768, X2 20MHz

Commit message: power, yo
Parts:
- BT1: BOM (none) -> DIST DIGIKEY BU2032SM-HD-GCT-ND
Changed lines of the file:
@@
 Connection ~ 4900 2100
 $Comp
-L GND #PWR155
+L GND #PWR158
 U 1 1 57981F37
 P 4900 2200
-F 0 "#PWR155" H 4900 2200 30  0001 C CNN
+F 0 "#PWR158" H 4900 2200 30  0001 C CNN
 F 1 "GND" H 4900 2130 30  0001 C CNN
 F 2 "" H 4900 2200 60  0000 C CNN
@@
 	6700 1500 6700 1600
 $Comp
-L GND #PWR158
+L GND #PWR160
 U 1 1 57983039
 P 6850 1700
-F 0 "#PWR158" H 6850 1700 30  0001 C CNN
+F 0 "#PWR160" H 6850 1700 30  0001 C CNN
 F 1 "GND" H 6850 1630 30  0001 C CNN
 F 2 "" H 6850 1700 60  0000 C CNN
@@
 Connection ~ 2100 1500
 $Comp
-L GND #PWR145
+L GND #PWR148
 U 1 1 57985104
 P 2100 1850
-F 0 "#PWR145" H 2100 1850 30  0001 C CNN
+F 0 "#PWR148" H 2100 1850 30  0001 C CNN
 F 1 "GND" H 2100 1780 30  0001 C CNN
 F 2 "" H 2100 1850 60  0000 C CNN
@@
 	2100 1850 2100 1800
 $Comp
-L GND #PWR146
+L GND #PWR149
 U 1 1 57985148
 P 2450 1850
-F 0 "#PWR146" H 2450 1850 30  0001 C CNN
+F 0 "#PWR149" H 2450 1850 30  0001 C CNN
 F 1 "GND" H 2450 1780 30  0001 C CNN
 F 2 "" H 2450 1850 60  0000 C CNN
@@
 	2450 1850 2450 1800
 $Comp
-L GND #PWR147
+L GND #PWR150
 U 1 1 5798515D
 P 2800 1850
-F 0 "#PWR147" H 2800 1850 30  0001 C CNN
+F 0 "#PWR150" H 2800 1850 30  0001 C CNN
 F 1 "GND" H 2800 1780 30  0001 C CNN
 F 2 "" H 2800 1850 60  0000 C CNN
@@
 	2800 1850 2800 1800
 $Comp
-L GND #PWR149
+L GND #PWR152
 U 1 1 57985164
 P 3150 1850
-F 0 "#PWR149" H 3150 1850 30  0001 C CNN
+F 0 "#PWR152" H 3150 1850 30  0001 C CNN
 F 1 "GND" H 3150 1780 30  0001 C CNN
 F 2 "" H 3150 1850 60  0000 C CNN
@@
 F 2 "" H 3800 1700 60  0000 C CNN
 F 3 "" H 3800 1700 60  0000 C CNN
+F 4 "DIST DIGIKEY BU2032SM-HD-GCT-ND" H 3800 1800 60  0001 C CNN "BOM"
 	1    3800 1800
 	1    0    0    -1
@@
 	3800 1600 3800 1700
 $Comp
-L GND #PWR151
+L GND #PWR154
 U 1 1 5798538F
 P 3800 2000
-F 0 "#PWR151" H 3800 2000 30  0001 C CNN
+F 0 "#PWR154" H 3800 2000 30  0001 C CNN
 F 1 "GND" H 3800 1930 30  0001 C CNN
 F 2 "" H 3800 2000 60  0000 C CNN
@@
 Connection ~ 4300 1600
 $Comp
-L GND #PWR152
+L GND #PWR155
 U 1 1 5798545A
 P 4300 2000
-F 0 "#PWR152" H 4300 2000 30  0001 C CNN
+F 0 "#PWR155" H 4300 2000 30  0001 C CNN
 F 1 "GND" H 4300 1930 30  0001 C CNN
 F 2 "" H 4300 2000 60  0000 C CNN
@@
 	6500 3200 6100 3200
 $Comp
-L GND #PWR157
+L GND #PWR159
 U 1 1 5798C21D
 P 6200 4100
-F 0 "#PWR157" H 6200 4100 30  0001 C CNN
+F 0 "#PWR159" H 6200 4100 30  0001 C CNN
 F 1 "GND" H 6200 4030 30  0001 C CNN
 F 2 "" H 6200 4100 60  0000 C CNN
@@
 	4300 3800 5100 3800
 $Comp
-L GND #PWR153
+L GND #PWR156
 U 1 1 5798C570
 P 4400 4000
-F 0 "#PWR153" H 4400 4000 30  0001 C CNN
+F 0 "#PWR156" H 4400 4000 30  0001 C CNN
 F 1 "GND" H 4400 3930 30  0001 C CNN
 F 2 "" H 4400 4000 60  0000 C CNN
@@
 	4400 3900 4300 3900
 $Comp
-L GND #PWR150
+L GND #PWR153
 U 1 1 5798C5E9
 P 3500 4100
-F 0 "#PWR150" H 3500 4100 30  0001 C CNN
+F 0 "#PWR153" H 3500 4100 30  0001 C CNN
 F 1 "GND" H 3500 4030 30  0001 C CNN
 F 2 "" H 3500 4100 60  0000 C CNN
@@
 Connection ~ 3100 3800
 $Comp
-L GND #PWR148
+L GND #PWR151
 U 1 1 5798C8CA
 P 3100 4150
-F 0 "#PWR148" H 3100 4150 30  0001 C CNN
+F 0 "#PWR151" H 3100 4150 30  0001 C CNN
 F 1 "GND" H 3100 4080 30  0001 C CNN
 F 2 "" H 3100 4150 60  0000 C CNN
@@
 Connection ~ 4600 3800
 $Comp
-L GND #PWR154
+L GND #PWR157
 U 1 1 5798C9F9
 P 4600 4150
-F 0 "#PWR154" H 4600 4150 30  0001 C CNN
+F 0 "#PWR157" H 4600 4150 30  0001 C CNN
 F 1 "GND" H 4600 4080 30  0001 C CNN
 F 2 "" H 4600 4150 60  0000 C CNN

Commit message: TODO: learn to write good commit messages
Parts:
- added C123, C124: 1u, IPC7351-Nominal:CAPC1005X55, symbol C-0402
- added U7, U8: LM75BDP, IPC7351-Nominal:SOP65P490X110-8, symbol LM75BDP
Connections:
- net GND: now also C123.2, C124.2, U7.4 (GND), U7.5 (A2), U7.6 (A1), U7.7 (A0), U8.4 (GND), U8.5 (A2), U8.6 (A1)
- net P3V3_AUX: now also C123.1, C124.1, U7.8 (V+), U8.7 (A0), U8.8 (V+)
- net SCL renamed SCL_S0
- net SCL_S0: now also U7.2 (SCL), U8.2 (SCL); no longer U3.6 (SCL)
- net SDA renamed SDA_S0
- net SDA_S0: now also U7.1 (SDA), U8.1 (SDA); no longer U3.5 (SDA)
- new net SCL_S5: U3.6 (SCL)
- new net SDA_S5: U3.5 (SDA)
- no-connect marks 2 -> 4
Changed lines of the file:
@@
 LIBS:semi-diode-Panasonic
 LIBS:Murata
+LIBS:semi-trans-Panasonic
 LIBS:c4puter-cache
 EELAYER 25 0
@@
 $EndComp
 Text HLabel 1600 2200 0    50   BiDi ~ 0
-SDA
+SDA_S5
 Text HLabel 1600 2300 0    50   Input ~ 0
-SCL
+SCL_S5
 Wire Wire Line
 	1600 2300 4800 2300
@@
 Connection ~ 4900 2100
 $Comp
-L GND #PWR158
+L GND #PWR176
 U 1 1 57981F37
 P 4900 2200
-F 0 "#PWR158" H 4900 2200 30  0001 C CNN
+F 0 "#PWR176" H 4900 2200 30  0001 C CNN
 F 1 "GND" H 4900 2130 30  0001 C CNN
 F 2 "" H 4900 2200 60  0000 C CNN
@@
 	6700 1500 6700 1600
 $Comp
-L GND #PWR160
+L GND #PWR180
 U 1 1 57983039
 P 6850 1700
-F 0 "#PWR160" H 6850 1700 30  0001 C CNN
+F 0 "#PWR180" H 6850 1700 30  0001 C CNN
 F 1 "GND" H 6850 1630 30  0001 C CNN
 F 2 "" H 6850 1700 60  0000 C CNN
@@
 Connection ~ 2100 1500
 $Comp
-L GND #PWR148
+L GND #PWR164
 U 1 1 57985104
 P 2100 1850
-F 0 "#PWR148" H 2100 1850 30  0001 C CNN
+F 0 "#PWR164" H 2100 1850 30  0001 C CNN
 F 1 "GND" H 2100 1780 30  0001 C CNN
 F 2 "" H 2100 1850 60  0000 C CNN
@@
 	2100 1850 2100 1800
 $Comp
-L GND #PWR149
+L GND #PWR165
 U 1 1 57985148
 P 2450 1850
-F 0 "#PWR149" H 2450 1850 30  0001 C CNN
+F 0 "#PWR165" H 2450 1850 30  0001 C CNN
 F 1 "GND" H 2450 1780 30  0001 C CNN
 F 2 "" H 2450 1850 60  0000 C CNN
@@
 	2450 1850 2450 1800
 $Comp
-L GND #PWR150
+L GND #PWR166
 U 1 1 5798515D
 P 2800 1850
-F 0 "#PWR150" H 2800 1850 30  0001 C CNN
+F 0 "#PWR166" H 2800 1850 30  0001 C CNN
 F 1 "GND" H 2800 1780 30  0001 C CNN
 F 2 "" H 2800 1850 60  0000 C CNN
@@
 	2800 1850 2800 1800
 $Comp
-L GND #PWR152
+L GND #PWR168
 U 1 1 57985164
 P 3150 1850
-F 0 "#PWR152" H 3150 1850 30  0001 C CNN
+F 0 "#PWR168" H 3150 1850 30  0001 C CNN
 F 1 "GND" H 3150 1780 30  0001 C CNN
 F 2 "" H 3150 1850 60  0000 C CNN
@@
 	3800 1600 3800 1700
 $Comp
-L GND #PWR154
+L GND #PWR170
 U 1 1 5798538F
 P 3800 2000
-F 0 "#PWR154" H 3800 2000 30  0001 C CNN
+F 0 "#PWR170" H 3800 2000 30  0001 C CNN
 F 1 "GND" H 3800 1930 30  0001 C CNN
 F 2 "" H 3800 2000 60  0000 C CNN
@@
 Connection ~ 4300 1600
 $Comp
-L GND #PWR155
+L GND #PWR171
 U 1 1 5798545A
 P 4300 2000
-F 0 "#PWR155" H 4300 2000 30  0001 C CNN
+F 0 "#PWR171" H 4300 2000 30  0001 C CNN
 F 1 "GND" H 4300 1930 30  0001 C CNN
 F 2 "" H 4300 2000 60  0000 C CNN
@@
 	6500 3200 6100 3200
 $Comp
-L GND #PWR159
+L GND #PWR179
 U 1 1 5798C21D
 P 6200 4100
-F 0 "#PWR159" H 6200 4100 30  0001 C CNN
+F 0 "#PWR179" H 6200 4100 30  0001 C CNN
 F 1 "GND" H 6200 4030 30  0001 C CNN
 F 2 "" H 6200 4100 60  0000 C CNN
@@
 	4500 3000 4600 3000
 Wire Wire Line
-	5100 3400 4100 3400
-Wire Wire Line
-	4100 3400 4100 2200
-Connection ~ 4100 2200
-Wire Wire Line
-	5100 3500 4000 3500
-Wire Wire Line
-	4000 3500 4000 2300
-Connection ~ 4000 2300
+	2400 3400 5100 3400
+Wire Wire Line
+	2300 3500 5100 3500
 NoConn ~ 5100 3650
 $Comp
@@
 	4300 3800 5100 3800
 $Comp
-L GND #PWR156
+L GND #PWR172
 U 1 1 5798C570
 P 4400 4000
-F 0 "#PWR156" H 4400 4000 30  0001 C CNN
+F 0 "#PWR172" H 4400 4000 30  0001 C CNN
 F 1 "GND" H 4400 3930 30  0001 C CNN
 F 2 "" H 4400 4000 60  0000 C CNN
@@
 	4400 3900 4300 3900
 $Comp
-L GND #PWR153
+L GND #PWR169
 U 1 1 5798C5E9
 P 3500 4100
-F 0 "#PWR153" H 3500 4100 30  0001 C CNN
+F 0 "#PWR169" H 3500 4100 30  0001 C CNN
 F 1 "GND" H 3500 4030 30  0001 C CNN
 F 2 "" H 3500 4100 60  0000 C CNN
@@
 Connection ~ 3100 3800
 $Comp
-L GND #PWR151
+L GND #PWR167
 U 1 1 5798C8CA
 P 3100 4150
-F 0 "#PWR151" H 3100 4150 30  0001 C CNN
+F 0 "#PWR167" H 3100 4150 30  0001 C CNN
 F 1 "GND" H 3100 4080 30  0001 C CNN
 F 2 "" H 3100 4150 60  0000 C CNN
@@
 Connection ~ 4600 3800
 $Comp
-L GND #PWR157
+L GND #PWR173
 U 1 1 5798C9F9
 P 4600 4150
-F 0 "#PWR157" H 4600 4150 30  0001 C CNN
+F 0 "#PWR173" H 4600 4150 30  0001 C CNN
 F 1 "GND" H 4600 4080 30  0001 C CNN
 F 2 "" H 4600 4150 60  0000 C CNN
@@
 Wire Wire Line
 	5000 4300 5000 3900
+$Comp
+L LM75BDP U7
+U 1 1 579F4ACE
+P 5600 4800
+F 0 "U7" H 5600 5067 50  0000 C CNN
+F 1 "LM75BDP" H 5600 4976 50  0000 C CNN
+F 2 "IPC7351-Nominal:SOP65P490X110-8" H 5600 4000 50  0001 C CNN
+F 3 "http://www.nxp.com/documents/data_sheet/LM75B.pdf" H 5600 3800 50  0001 C CNN
+F 4 "IC NXP LM75BDP" H 5600 3900 50  0001 C CNN "BOM"
+	1    5600 4800
+	1    0    0    -1
+$EndComp
+Text GLabel 4700 4800 0    50   Input ~ 0
+P3V3_AUX
+Wire Wire Line
+	4700 4800 5200 4800
+Text HLabel 1600 2500 0    50   BiDi ~ 0
+SDA_S0
+Text HLabel 1600 2600 0    50   Input ~ 0
+SCL_S0
+Wire Wire Line
+	1600 2500 2400 2500
+Wire Wire Line
+	2400 2500 2400 6000
+Wire Wire Line
+	2300 2600 2300 6100
+Wire Wire Line
+	2300 2600 1600 2600
+Wire Wire Line
+	2400 4900 5200 4900
+Connection ~ 2400 3400
+Wire Wire Line
+	2300 5000 5200 5000
+Connection ~ 2300 3500
+$Comp
+L GND #PWR177
+U 1 1 579F4E8E
+P 5100 5500
+F 0 "#PWR177" H 5100 5500 30  0001 C CNN
+F 1 "GND" H 5100 5430 30  0001 C CNN
+F 2 "" H 5100 5500 60  0000 C CNN
+F 3 "" H 5100 5500 60  0000 C CNN
+	1    5100 5500
+	1    0    0    -1
+$EndComp
+Wire Wire Line
+	5100 5500 5100 5100
+Wire Wire Line
+	5100 5100 5200 5100
+Wire Wire Line
+	5200 5200 5100 5200
+Connection ~ 5100 5200
+Wire Wire Line
+	5200 5300 5100 5300
+Connection ~ 5100 5300
+Wire Wire Line
+	5200 5400 5100 5400
+Connection ~ 5100 5400
+NoConn ~ 6000 4800
+$Comp
+L LM75BDP U8
+U 1 1 579F50E6
+P 5600 5900
+F 0 "U8" H 5600 6167 50  0000 C CNN
+F 1 "LM75BDP" H 5600 6076 50  0000 C CNN
+F 2 "IPC7351-Nominal:SOP65P490X110-8" H 5600 5100 50  0001 C CNN
+F 3 "http://www.nxp.com/documents/data_sheet/LM75B.pdf" H 5600 4900 50  0001 C CNN
+F 4 "IC NXP LM75BDP" H 5600 5000 50  0001 C CNN "BOM"
+	1    5600 5900
+	1    0    0    -1
+$EndComp
+NoConn ~ 6000 5900
+Text GLabel 4700 5900 0    50   Input ~ 0
+P3V3_AUX
+Wire Wire Line
+	4700 5900 5200 5900
+Wire Wire Line
+	2400 6000 5200 6000
+Connection ~ 2400 4900
+Wire Wire Line
+	2300 6100 5200 6100
+Connection ~ 2300 5000
+Wire Wire Line
+	5200 6300 5100 6300
+Wire Wire Line
+	5100 6300 5100 6600
+$Comp
+L GND #PWR178
+U 1 1 579F532E
+P 5100 6600
+F 0 "#PWR178" H 5100 6600 30  0001 C CNN
+F 1 "GND" H 5100 6530 30  0001 C CNN
+F 2 "" H 5100 6600 60  0000 C CNN
+F 3 "" H 5100 6600 60  0000 C CNN
+	1    5100 6600
+	1    0    0    -1
+$EndComp
+Wire Wire Line
+	5200 6400 5100 6400
+Connection ~ 5100 6400
+Wire Wire Line
+	5200 6500 5100 6500
+Connection ~ 5100 6500
+Wire Wire Line
+	5200 6200 5100 6200
+Wire Wire Line
+	5100 6200 5100 5900
+Connection ~ 5100 5900
+$Comp
+L C-0402 C?
+U 1 1 579F5ED1
+P 4800 5200
+AR Path="/5765A5BA/579F5ED1" Ref="C?"  Part="1"
+AR Path="/5765B2E6/579F5ED1" Ref="C?"  Part="1"
+AR Path="/57981212/579F5ED1" Ref="C123"  Part="1"
+F 0 "C123" H 4913 5246 50  0000 L CNN
+F 1 "1u" H 4913 5155 50  0000 L CNN
+F 2 "IPC7351-Nominal:CAPC1005X55" H 4800 5200 50  0001 C CNN
+F 3 "http://psearch.en.murata.com/capacitor/product/GRM155C80J105KE15%23.html" H 4790 5175 60  0001 C CNN
+F 4 "DIST DIGIKEY 490-6281-1-ND" H 5600 5750 60  0001 C CNN "BOM"
+	1    4800 5200
+	1    0    0    -1
+$EndComp
+Wire Wire Line
+	4800 5100 4800 4800
+Connection ~ 4800 4800
+$Comp
+L GND #PWR174
+U 1 1 579F5F9F
+P 4800 5400
+F 0 "#PWR174" H 4800 5400 30  0001 C CNN
+F 1 "GND" H 4800 5330 30  0001 C CNN
+F 2 "" H 4800 5400 60  0000 C CNN
+F 3 "" H 4800 5400 60  0000 C CNN
+	1    4800 5400
+	1    0    0    -1
+$EndComp
+Wire Wire Line
+	4800 5400 4800 5300
+$Comp
+L C-0402 C?
+U 1 1 579F605F
+P 4800 6300
+AR Path="/5765A5BA/579F605F" Ref="C?"  Part="1"
+AR Path="/5765B2E6/579F605F" Ref="C?"  Part="1"
+AR Path="/57981212/579F605F" Ref="C124"  Part="1"
+F 0 "C124" H 4913 6346 50  0000 L CNN
+F 1 "1u" H 4913 6255 50  0000 L CNN
+F 2 "IPC7351-Nominal:CAPC1005X55" H 4800 6300 50  0001 C CNN
+F 3 "http://psearch.en.murata.com/capacitor/product/GRM155C80J105KE15%23.html" H 4790 6275 60  0001 C CNN
+F 4 "DIST DIGIKEY 490-6281-1-ND" H 5600 6850 60  0001 C CNN "BOM"
+	1    4800 6300
+	1    0    0    -1
+$EndComp
+Wire Wire Line
+	4800 6200 4800 5900
+Connection ~ 4800 5900
+$Comp
+L GND #PWR175
+U 1 1 579F6133
+P 4800 6500
+F 0 "#PWR175" H 4800 6500 30  0001 C CNN
+F 1 "GND" H 4800 6430 30  0001 C CNN
+F 2 "" H 4800 6500 60  0000 C CNN
+F 3 "" H 4800 6500 60  0000 C CNN
+	1    4800 6500
+	1    0    0    -1
+$EndComp
+Wire Wire Line
+	4800 6500 4800 6400
 $EndSCHEMATC
