File: c4puter.sch (KiCad schematic (older format))
At the start: 26 parts, among them J7 19V 3A, J9 PANEL, Q1 AOD4189, Q2 AOD4189, SW1 POWER, SW2 SW

Commit message: Tidy up EC sheet
Parts:
- added J10: RS232, symbol CONN-100MIL-M-1x9
- added J8: DEBUG, conn-fci:CONN-10118194-0001LF-FCI, symbol CONN-10118194-0001LF-UUSB-B
- added SW3: SW-DIP-4, dip-sip:DIP-8, symbol SW-DIP-4
Connections:
- net labels added: RSCTS, RSDCD, RSDSR, RSDTR, RSRD, RSRI, RSRTS, RSTD, USB_VBUS, XUSB_D+, XUSB_D-
- wire segments 169 -> 195
- no-connect marks 0 -> 1
Changed lines of the file:
@@
 F32 "~PCIPME" I L 5200 5100 50
 F33 "PCIM66EN" I L 5200 5400 50
+F34 "RS232_TX" O L 5200 6300 50
+F35 "RS232_RX" I L 5200 6400 50
+F36 "RS232_RTS" O L 5200 6500 50
+F37 "RS232_CTS" I L 5200 6600 50
+F38 "USB_VBUS" I L 5200 6800 50
+F39 "XUSB_D-" B L 5200 6900 50
+F40 "XUSB_D+" B L 5200 7000 50
 $EndSheet
 Wire Wire Line
@@
 Wire Wire Line
 	12600 1800 11900 1800
+$Comp
+L CONN-100MIL-M-1x9 J?
+U 1 1 57A95B37
+P 1100 4600
+AR Path="/5765CB89/57A95B37" Ref="J?"  Part="1"
+AR Path="/57A95B37" Ref="J10"  Part="1"
+F 0 "J10" H 1219 4245 50  0000 L CNN
+F 1 "RS232" H 1219 4154 50  0000 L CNN
+F 2 "" H 1100 4600 50  0001 C CNN
+F 3 "" H 1100 4600 50  0000 C CNN
+	1    1100 4600
+	-1   0    0    -1
+$EndComp
+Text Label 1600 4600 2    50   ~ 0
+RSDCD
+Text Label 1600 4700 2    50   ~ 0
+RSRD
+Text Label 1600 4800 2    50   ~ 0
+RSTD
+Text Label 1600 4900 2    50   ~ 0
+RSDTR
+$Comp
+L GND #PWR?
+U 1 1 57A95B42
+P 1250 5000
+AR Path="/5765CB89/57A95B42" Ref="#PWR?"  Part="1"
+AR Path="/57A95B42" Ref="#PWR?"  Part="1"
+F 0 "#PWR?" H 1250 5000 30  0001 C CNN
+F 1 "GND" H 1250 4930 30  0001 C CNN
+F 2 "" H 1250 5000 60  0000 C CNN
+F 3 "" H 1250 5000 60  0000 C CNN
+	1    1250 5000
+	0    -1   -1   0
+$EndComp
+Text Label 1600 5100 2    50   ~ 0
+RSDSR
+Text Label 1600 5200 2    50   ~ 0
+RSRTS
+Text Label 1600 5300 2    50   ~ 0
+RSCTS
+Text Label 1600 5400 2    50   ~ 0
+RSRI
+Wire Wire Line
+	1600 4600 1150 4600
+Wire Wire Line
+	1150 4800 1600 4800
+Wire Wire Line
+	1150 4700 1600 4700
+Wire Wire Line
+	1250 5000 1150 5000
+Wire Wire Line
+	1600 4900 1150 4900
+Wire Wire Line
+	1600 5100 1150 5100
+Wire Wire Line
+	1150 5200 1600 5200
+Wire Wire Line
+	1150 5300 1600 5300
+Wire Wire Line
+	1600 5400 1150 5400
+Text Label 4700 6400 0    50   ~ 0
+RSRD
+Wire Wire Line
+	4700 6400 5200 6400
+Text Label 4700 6300 0    50   ~ 0
+RSTD
+Wire Wire Line
+	4700 6300 5200 6300
+Text Label 4700 6500 0    50   ~ 0
+RSRTS
+Wire Wire Line
+	4700 6500 5200 6500
+Text Label 4700 6600 0    50   ~ 0
+RSCTS
+Wire Wire Line
+	4700 6600 5200 6600
+$Comp
+L CONN-10118194-0001LF-UUSB-B J?
+U 1 1 57A9F4F6
+P 1100 3900
+AR Path="/5765CB89/57A9F4F6" Ref="J?"  Part="1"
+AR Path="/57A9F4F6" Ref="J8"  Part="1"
+F 0 "J8" H 1277 3920 50  0000 L CNN
+F 1 "DEBUG" H 1277 3829 50  0000 L CNN
+F 2 "conn-fci:CONN-10118194-0001LF-FCI" H 1100 3900 50  0001 C CNN
+F 3 "" H 1000 4100 50  0000 C CNN
+F 4 "DIST DIGIKEY 609-4618-1-ND" H 1600 4800 50  0001 C CNN "BOM"
+	1    1100 3900
+	-1   0    0    -1
+$EndComp
+Wire Wire Line
+	1300 4100 1400 4100
+Wire Wire Line
+	1400 4100 1400 4300
+$Comp
+L GND #PWR?
+U 1 1 57AA1CEB
+P 1400 4300
+F 0 "#PWR?" H 1400 4300 30  0001 C CNN
+F 1 "GND" H 1400 4230 30  0001 C CNN
+F 2 "" H 1400 4300 60  0000 C CNN
+F 3 "" H 1400 4300 60  0000 C CNN
+	1    1400 4300
+	1    0    0    -1
+$EndComp
+Text Label 4700 6900 0    50   ~ 0
+XUSB_D-
+Text Label 4700 7000 0    50   ~ 0
+XUSB_D+
+Wire Wire Line
+	4700 7000 5200 7000
+Wire Wire Line
+	5200 6900 4700 6900
+Text Label 4700 6800 0    50   ~ 0
+USB_VBUS
+Wire Wire Line
+	4700 6800 5200 6800
+Text Label 1700 3700 2    50   ~ 0
+USB_VBUS
+Wire Wire Line
+	1700 3700 1300 3700
+Text Label 1700 3800 2    50   ~ 0
+XUSB_D-
+Wire Wire Line
+	1300 3800 1700 3800
+Text Label 1700 3900 2    50   ~ 0
+XUSB_D+
+Wire Wire Line
+	1700 3900 1300 3900
+NoConn ~ 1300 4000
+$Comp
+L SW-DIP-4 SW3
+U 1 1 57AA9ABF
+P 1300 2900
+F 0 "SW3" H 1300 3167 50  0000 C CNN
+F 1 "SW-DIP-4" H 1300 3076 50  0000 C CNN
+F 2 "dip-sip:DIP-8" H 1300 2400 50  0001 C CNN
+F 3 "" H 1300 2800 50  0001 C CNN
+	1    1300 2900
+	1    0    0    -1
+$EndComp
+$Comp
+L GND #PWR?
+U 1 1 57AA9AC6
+P 900 3300
+AR Path="/5765CB89/57AA9AC6" Ref="#PWR?"  Part="1"
+AR Path="/57AA9AC6" Ref="#PWR?"  Part="1"
+F 0 "#PWR?" H 900 3300 30  0001 C CNN
+F 1 "GND" H 900 3230 30  0001 C CNN
+F 2 "" H 900 3300 60  0000 C CNN
+F 3 "" H 900 3300 60  0000 C CNN
+	1    900  3300
+	1    0    0    -1
+$EndComp
+Wire Wire Line
+	1000 2900 900  2900
+Wire Wire Line
+	900  2900 900  3300
+Wire Wire Line
+	1000 3200 900  3200
+Connection ~ 900  3200
+Wire Wire Line
+	1000 3100 900  3100
+Connection ~ 900  3100
+Wire Wire Line
+	1000 3000 900  3000
+Connection ~ 900  3000
 $EndSCHEMATC
