File: LIMB.sch (KiCad schematic (older format))
At the start: 50 parts, among them J2 MICROSD, J6 DEBUG, M1 FAN-4PIN, Q12 FK3303010L, Q13 FK3303010L, Q20 FK3303010L, Q21 FK3303010L, Q3 IRLML6402, U10 MAX3232PW, U11 NUF2042XV6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

Commit message: Connect SDRAM EVENT# line
Connections:
- net A0 renamed ~SDRAM_EVENT
Changed lines of the file:
@@
 $Descr B 17000 11000
 encoding utf-8
-Sheet 10 10
+Sheet 9 10
 Title "Local Integrated Management Bits"
 Date "2016-08-07"
@@
 	1    0    0    -1
 $EndComp
-Text Label 3600 3100 0    50   ~ 0
-A0
 Text Label 3600 3800 0    50   ~ 0
 A7
@@
 	3600 5700 3500 5700
 Wire Wire Line
-	3600 6200 3600 6700
+	3600 6200 3600 6300
+Wire Wire Line
+	3600 6300 3600 6400
+Wire Wire Line
+	3600 6400 3600 6500
+Wire Wire Line
+	3600 6500 3600 6600
+Wire Wire Line
+	3600 6600 3600 6700
 Wire Wire Line
 	3600 6200 3500 6200
@@
 Connection ~ 3600 6600
 Wire Wire Line
-	2100 1300 2300 1300
-Wire Wire Line
-	2200 1300 2200 1900
+	2100 1300 2200 1300
+Wire Wire Line
+	2200 1300 2300 1300
+Wire Wire Line
+	2200 1300 2200 1500
+Wire Wire Line
+	2200 1500 2200 1600
+Wire Wire Line
+	2200 1600 2200 1700
+Wire Wire Line
+	2200 1700 2200 1800
+Wire Wire Line
+	2200 1800 2200 1900
 Wire Wire Line
 	2200 1500 2300 1500
@@
 	9800 4000 9900 4000
 Wire Wire Line
-	8900 3800 9900 3800
+	8900 3800 9000 3800
+Wire Wire Line
+	9000 3800 9900 3800
 Wire Wire Line
 	9000 3900 9000 3800
@@
 	9000 4200 9000 4100
 Wire Wire Line
-	9800 4400 9800 4700
+	9800 4400 9800 4600
+Wire Wire Line
+	9800 4600 9800 4700
 Wire Wire Line
 	9900 4400 9800 4400
@@
 	1400 4800 2300 4800
 Wire Wire Line
-	2500 7500 4100 7500
-Wire Wire Line
-	2500 7600 4100 7600
+	2500 7500 2600 7500
+Wire Wire Line
+	2600 7500 4100 7500
+Wire Wire Line
+	2500 7600 3300 7600
+Wire Wire Line
+	3300 7600 4100 7600
 Wire Wire Line
 	4100 7700 2500 7700
 Wire Wire Line
-	2500 7800 4100 7800
-Wire Wire Line
-	2500 7900 4100 7900
+	2500 7800 2950 7800
+Wire Wire Line
+	2950 7800 4100 7800
+Wire Wire Line
+	2500 7900 3650 7900
+Wire Wire Line
+	3650 7900 4100 7900
 Wire Wire Line
 	2000 7900 2100 7900
 Wire Wire Line
-	2000 7600 2000 8000
+	2000 7600 2000 7700
+Wire Wire Line
+	2000 7700 2000 7900
+Wire Wire Line
+	2000 7900 2000 8000
 Wire Wire Line
 	2000 7700 2100 7700
@@
 	15000 5700 15000 5800
 Wire Wire Line
-	14350 6100 15300 6100
+	14350 6100 15000 6100
+Wire Wire Line
+	15000 6100 15300 6100
 Wire Wire Line
 	15000 6100 15000 6000
 Wire Wire Line
-	13950 6200 15300 6200
+	13950 6200 14700 6200
+Wire Wire Line
+	14700 6200 15300 6200
 Wire Wire Line
 	14700 6200 14700 6000
@@
 Connection ~ 14300 5700
 Wire Wire Line
-	13100 1300 15300 1300
+	13100 1300 13200 1300
+Wire Wire Line
+	13200 1300 14750 1300
+Wire Wire Line
+	14750 1300 15300 1300
 Wire Wire Line
 	14750 1400 14750 1300
@@
 	12050 3400 12100 3400
 Wire Wire Line
-	11600 2900 12400 2900
+	11600 2900 11800 2900
+Wire Wire Line
+	11800 2900 12400 2900
 Wire Wire Line
 	11800 2900 11800 3000
@@
 	12300 4100 12400 4100
 Wire Wire Line
-	13600 3800 15300 3800
+	13600 3800 14900 3800
+Wire Wire Line
+	14900 3800 15300 3800
 Connection ~ 14900 3800
 Wire Wire Line
@@
 	8600 2300 8500 2300
 Wire Wire Line
-	6400 1800 7100 1800
+	6400 1800 6900 1800
+Wire Wire Line
+	6900 1800 7100 1800
 Wire Wire Line
 	6400 1900 7100 1900
@@
 	15000 6600 15000 6650
 Wire Wire Line
-	14350 6900 15300 6900
+	14350 6900 15000 6900
+Wire Wire Line
+	15000 6900 15300 6900
 Wire Wire Line
 	15000 6900 15000 6850
@@
 	14700 6850 14700 7000
 Wire Wire Line
-	13950 7000 15300 7000
+	13950 7000 14700 7000
+Wire Wire Line
+	14700 7000 15300 7000
 Connection ~ 15000 6900
 Connection ~ 14700 7000
@@
 	2300 1400 2100 1400
 Wire Wire Line
-	2100 1400 2100 2400
+	2100 1400 2100 2000
+Wire Wire Line
+	2100 2000 2100 2100
+Wire Wire Line
+	2100 2100 2100 2200
+Wire Wire Line
+	2100 2200 2100 2300
+Wire Wire Line
+	2100 2300 2100 2400
 Wire Wire Line
 	2100 2000 2300 2000
@@
 	2000 7500 2000 7000
 Wire Wire Line
-	1900 7000 3650 7000
+	1900 7000 2000 7000
+Wire Wire Line
+	2000 7000 2600 7000
+Wire Wire Line
+	2600 7000 2950 7000
+Wire Wire Line
+	2950 7000 3300 7000
+Wire Wire Line
+	3300 7000 3650 7000
 Wire Wire Line
 	3300 7000 3300 7150
@@
 Connection ~ 2600 7000
 Wire Wire Line
-	13600 3700 15300 3700
+	13600 3700 14600 3700
+Wire Wire Line
+	14600 3700 15300 3700
 Wire Wire Line
 	14900 4200 14900 3800
 Wire Wire Line
-	13600 3900 15300 3900
-Wire Wire Line
-	13600 4000 15300 4000
+	13600 3900 14000 3900
+Wire Wire Line
+	14000 3900 15300 3900
+Wire Wire Line
+	13600 4000 14300 4000
+Wire Wire Line
+	14300 4000 15300 4000
 Wire Wire Line
 	15300 1900 14700 1900
@@
 	14800 2300 14700 2300
 Wire Wire Line
-	11800 5300 15300 5300
-Wire Wire Line
-	11800 5200 15300 5200
+	11800 5300 13100 5300
+Wire Wire Line
+	13100 5300 14700 5300
+Wire Wire Line
+	14700 5300 15300 5300
+Wire Wire Line
+	11800 5200 13200 5200
+Wire Wire Line
+	13200 5200 15000 5200
+Wire Wire Line
+	15000 5200 15300 5200
 Wire Wire Line
 	2000 3800 2300 3800
@@
 	2000 3900 2300 3900
 Wire Wire Line
-	6800 1300 7050 1300
+	6800 1300 6900 1300
+Wire Wire Line
+	6900 1300 7050 1300
 Connection ~ 6900 1300
 Connection ~ 9400 1300
 Wire Wire Line
-	9300 1300 9900 1300
-Wire Wire Line
-	14500 4800 15000 4800
+	9300 1300 9400 1300
+Wire Wire Line
+	9400 1300 9900 1300
+Wire Wire Line
+	14500 4800 14700 4800
+Wire Wire Line
+	14700 4800 15000 4800
 Wire Wire Line
 	15000 4800 15000 4900
@@
 Connection ~ 13900 5700
 Wire Wire Line
-	13800 5700 15000 5700
+	13800 5700 13900 5700
+Wire Wire Line
+	13900 5700 14300 5700
+Wire Wire Line
+	14300 5700 14700 5700
+Wire Wire Line
+	14700 5700 15000 5700
 Connection ~ 13900 6600
 Wire Wire Line
-	13800 6600 15000 6600
+	13800 6600 13900 6600
+Wire Wire Line
+	13900 6600 14300 6600
+Wire Wire Line
+	14300 6600 14700 6600
+Wire Wire Line
+	14700 6600 15000 6600
 Connection ~ 2000 7000
 Wire Wire Line
@@
 $EndComp
 Wire Wire Line
-	5500 3000 6400 3000
-Wire Wire Line
-	5500 3100 6400 3100
+	5500 3000 5900 3000
+Wire Wire Line
+	5900 3000 6400 3000
+Wire Wire Line
+	5500 3100 6200 3100
+Wire Wire Line
+	6200 3100 6400 3100
 Wire Wire Line
 	9100 3000 9100 3500
@@
 XMCDA3
 Wire Wire Line
-	5500 4100 6400 4100
+	5500 4100 5900 4100
+Wire Wire Line
+	5900 4100 6400 4100
 Wire Wire Line
 	8400 4100 8400 3700
@@
 	9300 4100 9300 5200
 Wire Wire Line
-	5500 5200 6400 5200
+	5500 5200 5900 5200
+Wire Wire Line
+	5900 5200 6400 5200
 Text Label 5500 5300 0    50   ~ 0
 MCDA1
 Wire Wire Line
-	5500 5300 6400 5300
+	5500 5300 6200 5300
+Wire Wire Line
+	6200 5300 6400 5300
 Text Label 9400 4100 0    50   ~ 0
 XMCDA0
@@
 	6700 2900 6600 2900
 Wire Wire Line
-	6600 2600 6600 5600
-Wire Wire Line
-	5850 2600 6600 2600
+	6600 2600 6600 2900
+Wire Wire Line
+	6600 2900 6600 3700
+Wire Wire Line
+	6600 3700 6600 4000
+Wire Wire Line
+	6600 4000 6600 4800
+Wire Wire Line
+	6600 4800 6600 5100
+Wire Wire Line
+	6600 5100 6600 5600
+Wire Wire Line
+	5850 2600 5900 2600
+Wire Wire Line
+	5900 2600 6200 2600
+Wire Wire Line
+	6200 2600 6600 2600
 Wire Wire Line
 	5900 2600 5900 2700
@@
 	6600 5100 6700 5100
 Wire Wire Line
-	5900 4800 6600 4800
+	5900 4800 6200 4800
+Wire Wire Line
+	6200 4800 6600 4800
 Wire Wire Line
 	5900 4800 5900 4900
@@
 $EndComp
 Wire Wire Line
-	6100 6000 9700 6000
+	6100 6000 6200 6000
+Wire Wire Line
+	6200 6000 9700 6000
 Wire Wire Line
 	6200 6000 6200 5900
@@
 P3V3_STBY
 Wire Wire Line
-	6900 6300 7300 6300
+	6900 6300 7150 6300
+Wire Wire Line
+	7150 6300 7300 6300
 $Comp
 L C-0402 C?
@@
 	7350 6600 7350 6400
 Wire Wire Line
-	6500 6600 7350 6600
+	6500 6600 7150 6600
+Wire Wire Line
+	7150 6600 7350 6600
 Text Label 6500 6600 0    50   ~ 0
 ~CARDEN
@@
 Text Label 2000 5500 0    50   ~ 0
 ~CARD
+Text HLabel 15300 9200 2    50   Input ~ 0
+~SDRAM_EVENT
+Text Label 11800 9200 0    50   ~ 0
+~SDRAM_EVENT
+Wire Wire Line
+	11800 9200 15300 9200
+Text Label 3600 3100 0    50   ~ 0
+~SDRAM_EVENT
 $EndSCHEMATC

Commit message: Add voltage reference
Parts:
- added C131: 1u, IPC7351-Nominal:CAPC1005X55, symbol C-0402
- added R131: 5k1, IPC7351-Nominal:RESC1005X40, symbol R-0402
- added U15: 2048mV, smd-semi:SC-70-5, symbol LM4040AvvDCK
Connections:
- net GND: now also C131.2, U15.1 (A)
- net at LIMB1.1 (ADVREF): now also C131.1, R131.2, U15.3 (K)
- net VREFEN: now reaches LIMB1.3 (PB0)
- net VREFEN: now also R131.1

Commit message: Set I2C pullups
Parts:
- R55, R8, R86, R9, R96, R97: value 5k1 -> 3k9; BOM RES SMD 5k1 1% [0402] -> RES SMD 3k9 1% [0402]
Changed lines of the file:
@@
 P 15000 5000
 F 0 "R8" H 15063 5046 50  0000 L CNN
-F 1 "5k1" H 15063 4955 50  0000 L CNN
+F 1 "3k9" H 15063 4955 50  0000 L CNN
 F 2 "IPC7351-Nominal:RESC1005X40" H 15000 5000 50  0001 C CNN
 F 3 "" H 15000 5050 60  0000 C CNN
-F 4 "RES SMD 5k1 1% [0402]" H 15750 5550 60  0001 C CNN "BOM"
+F 4 "RES SMD 3k9 1% [0402]" H 15750 5550 60  0001 C CNN "BOM"
 	1    15000 5000
 	-1   0    0    -1
@@
 P 14700 5000
 F 0 "R9" H 14763 5046 50  0000 L CNN
-F 1 "5k1" H 14763 4955 50  0000 L CNN
+F 1 "3k9" H 14763 4955 50  0000 L CNN
 F 2 "IPC7351-Nominal:RESC1005X40" H 14700 5000 50  0001 C CNN
 F 3 "" H 14700 5050 60  0000 C CNN
-F 4 "RES SMD 5k1 1% [0402]" H 15450 5550 60  0001 C CNN "BOM"
+F 4 "RES SMD 3k9 1% [0402]" H 15450 5550 60  0001 C CNN "BOM"
 	1    14700 5000
 	-1   0    0    -1
@@
 P 15000 5900
 F 0 "R55" H 15063 5946 50  0000 L CNN
-F 1 "5k1" H 15063 5855 50  0000 L CNN
+F 1 "3k9" H 15063 5855 50  0000 L CNN
 F 2 "IPC7351-Nominal:RESC1005X40" H 15000 5900 50  0001 C CNN
 F 3 "" H 15000 5950 60  0000 C CNN
-F 4 "RES SMD 5k1 1% [0402]" H 15750 6450 60  0001 C CNN "BOM"
+F 4 "RES SMD 3k9 1% [0402]" H 15750 6450 60  0001 C CNN "BOM"
 	1    15000 5900
 	-1   0    0    -1
@@
 P 14700 5900
 F 0 "R86" H 14763 5946 50  0000 L CNN
-F 1 "5k1" H 14763 5855 50  0000 L CNN
+F 1 "3k9" H 14763 5855 50  0000 L CNN
 F 2 "IPC7351-Nominal:RESC1005X40" H 14700 5900 50  0001 C CNN
 F 3 "" H 14700 5950 60  0000 C CNN
-F 4 "RES SMD 5k1 1% [0402]" H 15450 6450 60  0001 C CNN "BOM"
+F 4 "RES SMD 3k9 1% [0402]" H 15450 6450 60  0001 C CNN "BOM"
 	1    14700 5900
 	-1   0    0    -1
@@
 P 14700 6750
 F 0 "R97" H 14763 6796 50  0000 L CNN
-F 1 "5k1" H 14763 6705 50  0000 L CNN
+F 1 "3k9" H 14763 6705 50  0000 L CNN
 F 2 "IPC7351-Nominal:RESC1005X40" H 14700 6750 50  0001 C CNN
 F 3 "" H 14700 6800 60  0000 C CNN
-F 4 "RES SMD 5k1 1% [0402]" H 15450 7300 60  0001 C CNN "BOM"
+F 4 "RES SMD 3k9 1% [0402]" H 15450 7300 60  0001 C CNN "BOM"
 	1    14700 6750
 	-1   0    0    -1
@@
 P 15000 6750
 F 0 "R96" H 15063 6796 50  0000 L CNN
-F 1 "5k1" H 15063 6705 50  0000 L CNN
+F 1 "3k9" H 15063 6705 50  0000 L CNN
 F 2 "IPC7351-Nominal:RESC1005X40" H 15000 6750 50  0001 C CNN
 F 3 "" H 15000 6800 60  0000 C CNN
-F 4 "RES SMD 5k1 1% [0402]" H 15750 7300 60  0001 C CNN "BOM"
+F 4 "RES SMD 3k9 1% [0402]" H 15750 7300 60  0001 C CNN "BOM"
 	1    15000 6750
 	-1   0    0    -1

Commit message: Connect RTC alarm interrupt
Connections:
- net A7 renamed ~RTCINT
Changed lines of the file:
@@
 	1    0    0    -1
 $EndComp
-Text Label 3600 3800 0    50   ~ 0
-A7
 Text Label 3600 3900 0    50   ~ 0
 A8
@@
 Wire Wire Line
 	3800 4600 3500 4600
+Text HLabel 3600 3800 2    50   Input ~ 0
+~RTCINT
 $EndSCHEMATC

Commit message: IO expander for switches/buttons/LEDs
Connections:
- net A22 renamed ~PANELINT
Changed lines of the file:
@@
 Text Label 2000 3500 0    50   ~ 0
 A17
-Text Label 3600 3000 0    50   ~ 0
-A22
 Text Label 3600 1300 0    50   ~ 0
 D0
@@
 XOUT
 $Comp
-L GND #PWR187
+L GND #PWR188
 U 1 1 577EAB82
 P 3600 6700
-F 0 "#PWR187" H 3600 6700 30  0001 C CNN
+F 0 "#PWR188" H 3600 6700 30  0001 C CNN
 F 1 "GND" H 3600 6630 30  0001 C CNN
 F 2 "" H 3600 6700 60  0000 C CNN
@@
 $EndComp
 $Comp
-L GND #PWR195
+L GND #PWR196
 U 1 1 577EDCE7
 P 9800 4700
-F 0 "#PWR195" H 9800 4700 30  0001 C CNN
+F 0 "#PWR196" H 9800 4700 30  0001 C CNN
 F 1 "GND" H 9800 4630 30  0001 C CNN
 F 2 "" H 9800 4700 60  0000 C CNN
@@
 MCDA3
 $Comp
-L GND #PWR194
+L GND #PWR195
 U 1 1 577EDF0A
 P 9800 4000
-F 0 "#PWR194" H 9800 4000 30  0001 C CNN
+F 0 "#PWR195" H 9800 4000 30  0001 C CNN
 F 1 "GND" H 9800 3930 30  0001 C CNN
 F 2 "" H 9800 4000 60  0000 C CNN
@@
 P3V3_CARD
 $Comp
-L GND #PWR192
+L GND #PWR193
 U 1 1 577EEC84
 P 9000 4200
-F 0 "#PWR192" H 9000 4200 30  0001 C CNN
+F 0 "#PWR193" H 9000 4200 30  0001 C CNN
 F 1 "GND" H 9000 4130 30  0001 C CNN
 F 2 "" H 9000 4200 60  0000 C CNN
@@
 ~RST
 $Comp
-L GND #PWR186
+L GND #PWR187
 U 1 1 579F6A32
 P 2000 8000
-F 0 "#PWR186" H 2000 8000 30  0001 C CNN
+F 0 "#PWR187" H 2000 8000 30  0001 C CNN
 F 1 "GND" H 2000 7930 30  0001 C CNN
 F 2 "" H 2000 8000 60  0000 C CNN
@@
 Text GLabel 1900 7000 0    50   Input ~ 0
 P3V3_STBY
-Text HLabel 15300 8700 2    50   Input ~ 0
-BTN_PWR
-Text HLabel 15300 8800 2    50   Input ~ 0
-BTN_AUX
-Text HLabel 15300 8900 2    50   Output ~ 0
-LED_PWR
-Text HLabel 15300 9000 2    50   Output ~ 0
-LED_ACT
 $Comp
 L R-0402 R55
@@
 $EndComp
 $Comp
-L GND #PWR204
+L GND #PWR205
 U 1 1 57A172F2
 P 14750 1650
-F 0 "#PWR204" H 14750 1650 30  0001 C CNN
+F 0 "#PWR205" H 14750 1650 30  0001 C CNN
 F 1 "GND" H 14750 1580 30  0001 C CNN
 F 2 "" H 14750 1650 60  0000 C CNN
@@
 $EndComp
 $Comp
-L GND #PWR200
+L GND #PWR201
 U 1 1 57A1D8E5
 P 13950 3400
-F 0 "#PWR200" H 13950 3400 30  0001 C CNN
+F 0 "#PWR201" H 13950 3400 30  0001 C CNN
 F 1 "GND" H 13950 3330 30  0001 C CNN
 F 2 "" H 13950 3400 60  0000 C CNN
@@
 $EndComp
 $Comp
-L GND #PWR198
+L GND #PWR199
 U 1 1 57A1DE24
 P 12050 3400
-F 0 "#PWR198" H 12050 3400 30  0001 C CNN
+F 0 "#PWR199" H 12050 3400 30  0001 C CNN
 F 1 "GND" H 12050 3330 30  0001 C CNN
 F 2 "" H 12050 3400 60  0000 C CNN
@@
 $EndComp
 $Comp
-L GND #PWR197
+L GND #PWR198
 U 1 1 57A1E179
 P 11800 3250
-F 0 "#PWR197" H 11800 3250 30  0001 C CNN
+F 0 "#PWR198" H 11800 3250 30  0001 C CNN
 F 1 "GND" H 11800 3180 30  0001 C CNN
 F 2 "" H 11800 3250 60  0000 C CNN
@@
 P3V3_STBY
 $Comp
-L GND #PWR199
+L GND #PWR200
 U 1 1 57A1EEA9
 P 12300 4200
-F 0 "#PWR199" H 12300 4200 30  0001 C CNN
+F 0 "#PWR200" H 12300 4200 30  0001 C CNN
 F 1 "GND" H 12300 4130 30  0001 C CNN
 F 2 "" H 12300 4200 60  0000 C CNN
@@
 $EndComp
 $Comp
-L GND #PWR206
+L GND #PWR207
 U 1 1 57A22C9D
 P 14900 4450
-F 0 "#PWR206" H 14900 4450 30  0001 C CNN
+F 0 "#PWR207" H 14900 4450 30  0001 C CNN
 F 1 "GND" H 14900 4380 30  0001 C CNN
 F 2 "" H 14900 4450 60  0000 C CNN
@@
 $EndComp
 $Comp
-L GND #PWR203
+L GND #PWR204
 U 1 1 57A22E58
 P 14600 4450
-F 0 "#PWR203" H 14600 4450 30  0001 C CNN
+F 0 "#PWR204" H 14600 4450 30  0001 C CNN
 F 1 "GND" H 14600 4380 30  0001 C CNN
 F 2 "" H 14600 4450 60  0000 C CNN
@@
 $EndComp
 $Comp
-L GND #PWR202
+L GND #PWR203
 U 1 1 57A22FB0
 P 14300 4450
-F 0 "#PWR202" H 14300 4450 30  0001 C CNN
+F 0 "#PWR203" H 14300 4450 30  0001 C CNN
 F 1 "GND" H 14300 4380 30  0001 C CNN
 F 2 "" H 14300 4450 60  0000 C CNN
@@
 $EndComp
 $Comp
-L GND #PWR201
+L GND #PWR202
 U 1 1 57A23109
 P 14000 4450
-F 0 "#PWR201" H 14000 4450 30  0001 C CNN
+F 0 "#PWR202" H 14000 4450 30  0001 C CNN
 F 1 "GND" H 14000 4380 30  0001 C CNN
 F 2 "" H 14000 4450 60  0000 C CNN
@@
 $EndComp
 $Comp
-L GND #PWR193
+L GND #PWR194
 U 1 1 57A3FEDE
 P 9400 2100
-F 0 "#PWR193" H 9400 2100 30  0001 C CNN
+F 0 "#PWR194" H 9400 2100 30  0001 C CNN
 F 1 "GND" H 9400 2030 30  0001 C CNN
 F 2 "" H 9400 2100 60  0000 C CNN
@@
 $EndComp
 $Comp
-L GND #PWR191
+L GND #PWR192
 U 1 1 57A41BDC
 P 8600 2400
-F 0 "#PWR191" H 8600 2400 30  0001 C CNN
+F 0 "#PWR192" H 8600 2400 30  0001 C CNN
 F 1 "GND" H 8600 2330 30  0001 C CNN
 F 2 "" H 8600 2400 60  0000 C CNN
@@
 $EndComp
 $Comp
-L GND #PWR196
+L GND #PWR197
 U 1 1 57A49C3C
 P 9900 1750
-F 0 "#PWR196" H 9900 1750 30  0001 C CNN
+F 0 "#PWR197" H 9900 1750 30  0001 C CNN
 F 1 "GND" H 9900 1680 30  0001 C CNN
 F 2 "" H 9900 1750 60  0000 C CNN
@@
 XUSB_D+
 $Comp
-L GND #PWR205
+L GND #PWR206
 U 1 1 57AA14DB
 P 14800 2400
-F 0 "#PWR205" H 14800 2400 30  0001 C CNN
+F 0 "#PWR206" H 14800 2400 30  0001 C CNN
 F 1 "GND" H 14800 2330 30  0001 C CNN
 F 2 "" H 14800 2400 60  0000 C CNN
@@
 Connection ~ 5900 2600
 $Comp
-L GND #PWR188
+L GND #PWR189
 U 1 1 57A9C7D3
 P 8200 3550
-F 0 "#PWR188" H 8200 3550 30  0001 C CNN
+F 0 "#PWR189" H 8200 3550 30  0001 C CNN
 F 1 "GND" H 8200 3480 30  0001 C CNN
 F 2 "" H 8200 3550 60  0000 C CNN
@@
 	8200 3500 8100 3500
 $Comp
-L GND #PWR189
+L GND #PWR190
 U 1 1 57A9C9F3
 P 8200 4650
-F 0 "#PWR189" H 8200 4650 30  0001 C CNN
+F 0 "#PWR190" H 8200 4650 30  0001 C CNN
 F 1 "GND" H 8200 4580 30  0001 C CNN
 F 2 "" H 8200 4650 60  0000 C CNN
@@
 	8200 4600 8100 4600
 $Comp
-L GND #PWR190
+L GND #PWR191
 U 1 1 57A9CC0D
 P 8200 5750
-F 0 "#PWR190" H 8200 5750 30  0001 C CNN
+F 0 "#PWR191" H 8200 5750 30  0001 C CNN
 F 1 "GND" H 8200 5680 30  0001 C CNN
 F 2 "" H 8200 5750 60  0000 C CNN
@@
 Connection ~ 1150 3200
 $Comp
-L GND #PWR184
+L GND #PWR185
 U 1 1 57AAC080
 P 1150 3700
-F 0 "#PWR184" H 1150 3700 30  0001 C CNN
+F 0 "#PWR185" H 1150 3700 30  0001 C CNN
 F 1 "GND" H 1150 3630 30  0001 C CNN
 F 2 "" H 1150 3700 60  0000 C CNN
@@
 Connection ~ 1400 3200
 $Comp
-L GND #PWR185
+L GND #PWR186
 U 1 1 57AB076E
 P 1400 3700
-F 0 "#PWR185" H 1400 3700 30  0001 C CNN
+F 0 "#PWR186" H 1400 3700 30  0001 C CNN
 F 1 "GND" H 1400 3630 30  0001 C CNN
 F 2 "" H 1400 3700 60  0000 C CNN
@@
 Text HLabel 3600 3800 2    50   Input ~ 0
 ~RTCINT
+Text HLabel 15300 8600 2    50   Input ~ 0
+~PANELINT
+Wire Wire Line
+	15300 8600 11800 8600
+Text Label 11800 8600 0    50   ~ 0
+~PANELINT
+Text Label 3600 3000 0    50   ~ 0
+~PANELINT
 $EndSCHEMATC
