File: Power.sch (KiCad schematic (older format))
At the start: 75 parts, among them Q10 AOD514, Q11 AOD514, Q14 FK3303010L, Q15 FK3303010L, Q16 FK3303010L, Q17 FK3303010L, Q18 FK3303010L, Q4 FK3303010L, Q5 FK3303010L, Q6 FK3303010L, Q9 AOD417, U2 PCF8575, U6 RT9026GFP

Commit message: Squiggles! Silk!
Parts:
- renumbered C3 to C901, C4 to C902, C5 to C903, C6 to C904, C82 to C905, C34 to C906, C33 to C907, C56 to C908, C55 to C909, C110 to C910, C111 to C911, C112 to C912, C113 to C913, C114 to C914, E2 to E901, E1 to E902, JP1 to JP901, JP2 to JP902, JP3 to JP903, JP8 to JP904, JP9 to JP905, JP13 to JP906, JP10 to JP907, JP11 to JP908, JP12 to JP909, JP4 to JP910, JP6 to JP911, JP7 to JP912, Q6 to Q901, Q5 to Q902, Q4 to Q903, Q18 to Q904, Q17 to Q905, Q14 to Q906, Q15 to Q907, Q16 to Q908, Q9 to Q909, Q10 to Q910, Q11 to Q911, R59 to R901, R60 to R902, R61 to R903, R57 to R904, R68 to R905, R75 to R906, R76 to R907, R58 to R908, R114 to R909, R115 to R910, R63 to R911, R64 to R912, R69 to R913, R70 to R914, R65 to R915, R66 to R916, R67 to R917, R62 to R918, R77 to R919, R78 to R920, R79 to R921, R81 to R922, R82 to R923, R83 to R924, R84 to R925, R80 to R926, U2 to U901, U6 to U902, VREG2 to VREG901, VREG1 to VREG902, VRM1 to VRM901, W1 to W901, W2 to W902, W3 to W903, W4 to W904, W5 to W905

Commit message: Final BOM
Parts:
- E901, E902: value 100 -> 120; BOM BEAD SMD 100 @0MHz 1A [1812] -> BEAD SMD 120 1A [1812]
Changed lines of the file:
@@
 U 1 1 5791C29F
 P 8600 6900
-F 0 "E902" H 8600 7125 50  0000 C CNN
-F 1 "100" H 8600 7034 50  0000 C CNN
+F 0 "E902" H 8600 7150 50  0000 C CNN
+F 1 "120" H 8600 7050 50  0000 C CNN
 F 2 "IPC7351-Nominal:CAPC4532X220" H 8600 6800 50  0001 C CNN
 F 3 "" H 8600 6950 60  0000 C CNN
-F 4 "BEAD SMD 100 @0MHz 1A [1812]" H 8600 6700 60  0001 C CNN "BOM"
+F 4 "BEAD SMD 120 1A [1812]" H 8600 6700 60  0001 C CNN "BOM"
 	1    8600 6900
 	1    0    0    -1
@@
 U 1 1 5791EC24
 P 8600 5800
-F 0 "E901" H 8600 6025 50  0000 C CNN
-F 1 "100" H 8600 5934 50  0000 C CNN
+F 0 "E901" H 8600 6050 50  0000 C CNN
+F 1 "120" H 8600 5950 50  0000 C CNN
 F 2 "IPC7351-Nominal:CAPC4532X220" H 8600 5700 50  0001 C CNN
 F 3 "" H 8600 5850 60  0000 C CNN
-F 4 "BEAD SMD 100 @0MHz 1A [1812]" H 8600 5600 60  0001 C CNN "BOM"
+F 4 "BEAD SMD 120 1A [1812]" H 8600 5600 60  0001 C CNN "BOM"
 	1    8600 5800
 	1    0    0    -1

Commit message: Remove current sense resistors, add I2C debug header
Parts:
- removed JP901, JP902, JP903, JP904, JP905, JP906, JP907, JP908, JP909, JP910, JP911, JP912: JUMPER-SOLDER, conn-test:JUMPER-SOLDER-SMD, symbol JUMPER-SOLDER
- removed R920, R921, R923, R925: R001, manuf:VISHAY-WSL3637-LARGE, symbol R-VISHAY-WSL3637-LARGE
- removed R922, R924: R01, IPC7351-Nominal:RESC2012X50, symbol R-0805
- removed R926: R20, IPC7351-Nominal:RESC2012X50, symbol R-0805
- added JP902, JP903, JP905, JP909: 0R, IPC7351-Nominal:RESC3216X60, symbol R-1206
- added JP904, JP906, JP907, JP908, JP910, JP911, JP912: 0R, IPC7351-Nominal:RESC2012X50, symbol R-0805
- JP901: renamed from R919; value R01 -> 0R; BOM RES SMD R01 1% [0805] -> RES SMD 0R HighCurrent [0805]
Connections:
- wire segments 330 -> 470
- no-connect marks 11 -> 3
Other:
- moved on the sheet: JP901

Commit message: Add some test points
Parts:
- added TP901, TP902: VTT_S3, conn-test:TEST-SMD-SMALL, symbol TESTPOINT
Connections:
- net EN_V75: now also TP901.1
- net EN_V75REF: now also TP902.1

Commit message: Update for KiCad 5
Parts:
- C901, C902, C903, C904: symbol C-ALUM-8mm -> pasv-cap:C-ALUM-8mm
- C905, C906, C907, C908, C909, C910, C912: symbol C-0402 -> pasv-cap:C-0402
- C911, C913, C914: symbol C-0603 -> pasv-cap:C-0603
- E901, E902: symbol BEAD-1812 -> pasv-ind:BEAD-1812
- JP901, JP904, JP906, JP907, JP908, JP910, JP911, JP912: symbol R-0805 -> pasv-res:R-0805
- JP902, JP903, JP905, JP909: symbol R-1206 -> pasv-res:R-1206
- Q901, Q902, Q903, Q904, Q905, Q906, Q907, Q908: symbol FK3303010L -> semi-trans-Panasonic:FK3303010L
- Q909: symbol AOD417 -> semi-trans-AOS:AOD417
- Q910, Q911: symbol AOD514 -> semi-trans-AOS:AOD514
- R901, R902, R903, R904, R905, R906, R907, R908, R909, R910: symbol R-0402 -> pasv-res:R-0402
- R911, R912, R913, R914, R915, R916, R917, R918: symbol R-0603 -> pasv-res:R-0603
- TP901, TP902: symbol TESTPOINT -> pcb:TESTPOINT
- U901: symbol PCF8575 -> NXP:PCF8575
- U902: symbol RT9026GFP -> Richtek:RT9026GFP
- VREG901, VREG902: symbol OKX-T/5-W5N-C -> Murata:OKX-T_5-W5N-C
- VRM901: symbol CONN-10018783-10202TLF-PCIEx8 -> conn-fci:CONN-10018783-10202TLF-PCIEx8
- W901, W902, W903, W904, W905: symbol NET-TIE -> symbol:NET-TIE
