File: PCI.sch (KiCad schematic (older format))
At the start: 75 parts

Commit message: Squiggles! Silk!
Parts:
- renumbered C35 to C401, C36 to C402, C37 to C403, C38 to C404, C51 to C405, C71 to C406, C39 to C407, C40 to C408, C41 to C409, C42 to C410, C52 to C411, C72 to C412, C43 to C413, C44 to C414, C45 to C415, C46 to C416, C53 to C417, C73 to C418, C47 to C419, C48 to C420, C49 to C421, C50 to C422, C54 to C423, C74 to C424, C58 to C425, C60 to C426, C61 to C427, C62 to C428, C63 to C429, C67 to C430, C64 to C431, C68 to C432, C116 to C433, C117 to C434, C118 to C435, C65 to C436, C69 to C437, C119 to C438, C120 to C439, C121 to C440, C66 to C441, C70 to C442, R23 to R401, R24 to R402, R25 to R403, R26 to R404, R27 to R405, R28 to R406, R29 to R407, R127 to R408, R30 to R409, R31 to R410, R32 to R411, R41 to R412, R42 to R413, R128 to R414, R33 to R415, R34 to R416, R35 to R417, R43 to R418, R44 to R419, R129 to R420, R36 to R421, R37 to R422, R38 to R423, R45 to R424, R46 to R425, R49 to R426, R130 to R427, R47 to R428, R48 to R429

Commit message: Final BOM
Parts:
- removed R401, R402, R403, R404: 160, IPC7351-Nominal:RESC1005X40, symbol R-0402
- added R401, R402, R403, R404: 120, IPC7351-Nominal:RESC1608X50, symbol R-0603
- R408, R412, R413, R414, R418, R419, R420, R424, R425, R426, R427, R428, R429: value 5k1 -> 4k3; BOM RES SMD 5k1 1% [0402] -> RES SMD 4k3 [0402]
Connections:
- net AD16: now also R401.2
- net AD17: now also R402.2
- net AD18: now also R403.2
- net AD19: now also R404.2
- net IDSEL0: now also R401.1
- net IDSEL1: now also R402.1
- net IDSEL2: now also R403.1
- net IDSEL3: now also R404.1
Changed lines of the file:
@@
 P 14700 1200
 F 0 "R412" V 14500 1200 50  0000 C CNN
-F 1 "5k1" V 14591 1200 50  0000 C CNN
+F 1 "4k3" V 14591 1200 50  0000 C CNN
 F 2 "IPC7351-Nominal:RESC1005X40" H 14700 1200 50  0001 C CNN
 F 3 "" H 14700 1250 60  0000 C CNN
-F 4 "RES SMD 5k1 1% [0402]" H 15450 1750 60  0001 C CNN "BOM"
+F 4 "RES SMD 4k3 [0402]" H 15450 1750 60  0001 C CNN "BOM"
 	1    14700 1200
 	0    1    1    0
@@
 P 15000 1300
 F 0 "R418" V 14750 1300 50  0000 C CNN
-F 1 "5k1" V 14850 1300 50  0000 C CNN
+F 1 "4k3" V 14850 1300 50  0000 C CNN
 F 2 "IPC7351-Nominal:RESC1005X40" H 15000 1300 50  0001 C CNN
 F 3 "" H 15000 1350 60  0000 C CNN
-F 4 "RES SMD 5k1 1% [0402]" H 15750 1850 60  0001 C CNN "BOM"
+F 4 "RES SMD 4k3 [0402]" H 15750 1850 60  0001 C CNN "BOM"
 	1    15000 1300
 	0    1    1    0
@@
 P 15300 1400
 F 0 "R424" V 15050 1400 50  0000 C CNN
-F 1 "5k1" V 15150 1400 50  0000 C CNN
+F 1 "4k3" V 15150 1400 50  0000 C CNN
 F 2 "IPC7351-Nominal:RESC1005X40" H 15300 1400 50  0001 C CNN
 F 3 "" H 15300 1450 60  0000 C CNN
-F 4 "RES SMD 5k1 1% [0402]" H 16050 1950 60  0001 C CNN "BOM"
+F 4 "RES SMD 4k3 [0402]" H 16050 1950 60  0001 C CNN "BOM"
 	1    15300 1400
 	0    1    1    0
@@
 P 15600 1500
 F 0 "R428" V 15350 1500 50  0000 C CNN
-F 1 "5k1" V 15450 1500 50  0000 C CNN
+F 1 "4k3" V 15450 1500 50  0000 C CNN
 F 2 "IPC7351-Nominal:RESC1005X40" H 15600 1500 50  0001 C CNN
 F 3 "" H 15600 1550 60  0000 C CNN
-F 4 "RES SMD 5k1 1% [0402]" H 16350 2050 60  0001 C CNN "BOM"
+F 4 "RES SMD 4k3 [0402]" H 16350 2050 60  0001 C CNN "BOM"
 	1    15600 1500
 	0    1    1    0
@@
 P 14700 1600
 F 0 "R413" V 14450 1600 50  0000 C CNN
-F 1 "5k1" V 14550 1600 50  0000 C CNN
+F 1 "4k3" V 14550 1600 50  0000 C CNN
 F 2 "IPC7351-Nominal:RESC1005X40" H 14700 1600 50  0001 C CNN
 F 3 "" H 14700 1650 60  0000 C CNN
-F 4 "RES SMD 5k1 1% [0402]" H 15450 2150 60  0001 C CNN "BOM"
+F 4 "RES SMD 4k3 [0402]" H 15450 2150 60  0001 C CNN "BOM"
 	1    14700 1600
 	0    1    1    0
@@
 P 15000 1700
 F 0 "R419" V 14750 1700 50  0000 C CNN
-F 1 "5k1" V 14850 1700 50  0000 C CNN
+F 1 "4k3" V 14850 1700 50  0000 C CNN
 F 2 "IPC7351-Nominal:RESC1005X40" H 15000 1700 50  0001 C CNN
 F 3 "" H 15000 1750 60  0000 C CNN
-F 4 "RES SMD 5k1 1% [0402]" H 15750 2250 60  0001 C CNN "BOM"
+F 4 "RES SMD 4k3 [0402]" H 15750 2250 60  0001 C CNN "BOM"
 	1    15000 1700
 	0    1    1    0
@@
 P 15300 1800
 F 0 "R425" V 15050 1800 50  0000 C CNN
-F 1 "5k1" V 15150 1800 50  0000 C CNN
+F 1 "4k3" V 15150 1800 50  0000 C CNN
 F 2 "IPC7351-Nominal:RESC1005X40" H 15300 1800 50  0001 C CNN
 F 3 "" H 15300 1850 60  0000 C CNN
-F 4 "RES SMD 5k1 1% [0402]" H 16050 2350 60  0001 C CNN "BOM"
+F 4 "RES SMD 4k3 [0402]" H 16050 2350 60  0001 C CNN "BOM"
 	1    15300 1800
 	0    1    1    0
@@
 P 15600 1900
 F 0 "R429" V 15350 1900 50  0000 C CNN
-F 1 "5k1" V 15450 1900 50  0000 C CNN
+F 1 "4k3" V 15450 1900 50  0000 C CNN
 F 2 "IPC7351-Nominal:RESC1005X40" H 15600 1900 50  0001 C CNN
 F 3 "" H 15600 1950 60  0000 C CNN
-F 4 "RES SMD 5k1 1% [0402]" H 16350 2450 60  0001 C CNN "BOM"
+F 4 "RES SMD 4k3 [0402]" H 16350 2450 60  0001 C CNN "BOM"
 	1    15600 1900
 	0    1    1    0
@@
 P 15300 2700
 F 0 "R426" H 15237 2654 50  0000 R CNN
-F 1 "5k1" H 15237 2745 50  0000 R CNN
+F 1 "4k3" H 15237 2745 50  0000 R CNN
 F 2 "IPC7351-Nominal:RESC1005X40" H 15300 2700 50  0001 C CNN
 F 3 "" H 15300 2750 60  0000 C CNN
-F 4 "RES SMD 5k1 1% [0402]" H 16050 3250 60  0001 C CNN "BOM"
+F 4 "RES SMD 4k3 [0402]" H 16050 3250 60  0001 C CNN "BOM"
 	1    15300 2700
 	-1   0    0    1
@@
 	0    -1   -1   0
 $EndComp
-$Comp
-L R-0402 R401
-U 1 1 57A827BF
-P 2400 5200
-F 0 "R401" V 2200 5200 50  0000 C CNN
-F 1 "160" V 2291 5200 50  0000 C CNN
-F 2 "IPC7351-Nominal:RESC1005X40" H 2400 5200 50  0001 C CNN
-F 3 "" H 2400 5250 60  0000 C CNN
-F 4 "RES SMD 160 1% [0402]" H 3150 5750 60  0001 C CNN "BOM"
-	1    2400 5200
-	0    1    1    0
-$EndComp
-$Comp
-L R-0402 R402
-U 1 1 57A82D82
-P 5300 5200
-F 0 "R402" V 5100 5200 50  0000 C CNN
-F 1 "160" V 5191 5200 50  0000 C CNN
-F 2 "IPC7351-Nominal:RESC1005X40" H 5300 5200 50  0001 C CNN
-F 3 "" H 5300 5250 60  0000 C CNN
-F 4 "RES SMD 160 1% [0402]" H 6050 5750 60  0001 C CNN "BOM"
-	1    5300 5200
-	0    1    1    0
-$EndComp
-$Comp
-L R-0402 R403
-U 1 1 57A83095
-P 8100 5200
-F 0 "R403" V 7900 5200 50  0000 C CNN
-F 1 "160" V 7991 5200 50  0000 C CNN
-F 2 "IPC7351-Nominal:RESC1005X40" H 8100 5200 50  0001 C CNN
-F 3 "" H 8100 5250 60  0000 C CNN
-F 4 "RES SMD 160 1% [0402]" H 8850 5750 60  0001 C CNN "BOM"
-	1    8100 5200
-	0    1    1    0
-$EndComp
-$Comp
-L R-0402 R404
-U 1 1 57A8358C
-P 10900 5200
-F 0 "R404" V 10700 5200 50  0000 C CNN
-F 1 "160" V 10791 5200 50  0000 C CNN
-F 2 "IPC7351-Nominal:RESC1005X40" H 10900 5200 50  0001 C CNN
-F 3 "" H 10900 5250 60  0000 C CNN
-F 4 "RES SMD 160 1% [0402]" H 11650 5750 60  0001 C CNN "BOM"
-	1    10900 5200
-	0    1    1    0
-$EndComp
 Text GLabel 15200 4000 0    50   Input ~ 0
 P3V3_AUX
@@
 P 14500 4300
 F 0 "R408" V 14300 4300 50  0000 C CNN
-F 1 "5k1" V 14391 4300 50  0000 C CNN
+F 1 "4k3" V 14391 4300 50  0000 C CNN
 F 2 "IPC7351-Nominal:RESC1005X40" H 14500 4300 50  0001 C CNN
 F 3 "" H 14500 4350 60  0000 C CNN
-F 4 "RES SMD 5k1 1% [0402]" H 15250 4850 60  0001 C CNN "BOM"
+F 4 "RES SMD 4k3 [0402]" H 15250 4850 60  0001 C CNN "BOM"
 	1    14500 4300
 	0    1    1    0
@@
 P 14800 4400
 F 0 "R414" V 14550 4400 50  0000 C CNN
-F 1 "5k1" V 14650 4400 50  0000 C CNN
+F 1 "4k3" V 14650 4400 50  0000 C CNN
 F 2 "IPC7351-Nominal:RESC1005X40" H 14800 4400 50  0001 C CNN
 F 3 "" H 14800 4450 60  0000 C CNN
-F 4 "RES SMD 5k1 1% [0402]" H 15550 4950 60  0001 C CNN "BOM"
+F 4 "RES SMD 4k3 [0402]" H 15550 4950 60  0001 C CNN "BOM"
 	1    14800 4400
 	0    1    1    0
@@
 P 15100 4500
 F 0 "R420" V 14850 4500 50  0000 C CNN
-F 1 "5k1" V 14950 4500 50  0000 C CNN
+F 1 "4k3" V 14950 4500 50  0000 C CNN
 F 2 "IPC7351-Nominal:RESC1005X40" H 15100 4500 50  0001 C CNN
 F 3 "" H 15100 4550 60  0000 C CNN
-F 4 "RES SMD 5k1 1% [0402]" H 15850 5050 60  0001 C CNN "BOM"
+F 4 "RES SMD 4k3 [0402]" H 15850 5050 60  0001 C CNN "BOM"
 	1    15100 4500
 	0    1    1    0
@@
 P 15400 4600
 F 0 "R427" V 15508 4600 50  0000 C CNN
-F 1 "5k1" V 15599 4600 50  0000 C CNN
+F 1 "4k3" V 15599 4600 50  0000 C CNN
 F 2 "IPC7351-Nominal:RESC1005X40" H 15400 4600 50  0001 C CNN
 F 3 "" H 15400 4650 60  0000 C CNN
-F 4 "RES SMD 5k1 1% [0402]" H 16150 5150 60  0001 C CNN "BOM"
+F 4 "RES SMD 4k3 [0402]" H 16150 5150 60  0001 C CNN "BOM"
 	1    15400 4600
 	0    1    1    0
@@
 Wire Wire Line
 	15400 7200 15300 7200
+$Comp
+L R-0603 R401
+U 1 1 57B0D372
+P 2400 5200
+F 0 "R401" V 2200 5200 50  0000 C CNN
+F 1 "120" V 2291 5200 50  0000 C CNN
+F 2 "IPC7351-Nominal:RESC1608X50" H 2400 5200 50  0001 C CNN
+F 3 "" H 2400 5250 60  0000 C CNN
+F 4 "RES SMD 120 5% [0603]" H 3150 5750 60  0001 C CNN "BOM"
+	1    2400 5200
+	0    1    1    0
+$EndComp
+$Comp
+L R-0603 R402
+U 1 1 57B0D805
+P 5300 5200
+F 0 "R402" V 5100 5200 50  0000 C CNN
+F 1 "120" V 5191 5200 50  0000 C CNN
+F 2 "IPC7351-Nominal:RESC1608X50" H 5300 5200 50  0001 C CNN
+F 3 "" H 5300 5250 60  0000 C CNN
+F 4 "RES SMD 120 5% [0603]" H 6050 5750 60  0001 C CNN "BOM"
+	1    5300 5200
+	0    1    1    0
+$EndComp
+$Comp
+L R-0603 R403
+U 1 1 57B0DC5D
+P 8100 5200
+F 0 "R403" V 7900 5200 50  0000 C CNN
+F 1 "120" V 7991 5200 50  0000 C CNN
+F 2 "IPC7351-Nominal:RESC1608X50" H 8100 5200 50  0001 C CNN
+F 3 "" H 8100 5250 60  0000 C CNN
+F 4 "RES SMD 120 5% [0603]" H 8850 5750 60  0001 C CNN "BOM"
+	1    8100 5200
+	0    1    1    0
+$EndComp
+$Comp
+L R-0603 R404
+U 1 1 57B0E034
+P 10900 5200
+F 0 "R404" V 10700 5200 50  0000 C CNN
+F 1 "120" V 10791 5200 50  0000 C CNN
+F 2 "IPC7351-Nominal:RESC1608X50" H 10900 5200 50  0001 C CNN
+F 3 "" H 10900 5250 60  0000 C CNN
+F 4 "RES SMD 120 5% [0603]" H 11650 5750 60  0001 C CNN "BOM"
+	1    10900 5200
+	0    1    1    0
+$EndComp
 $EndSCHEMATC

Commit message: Tidy schematics and produce PDF
Other:
- moved on the sheet: C401, C402, C403, C404, C405, C406, C407, C408, C409, C410, C411, C412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

Commit message: Update for KiCad 5
Parts:
- C401, C402, C403, C404, C405, C406, C407, C408, C409, C410, C411, C412, C413, C414, C415, C416, C417, C418, C419, C420, C421, C422, C423, C424: symbol C-ALUM-6.3mm -> pasv-cap:C-ALUM-6.3mm
- C425, C426, C427, C428, C429, C430, C431, C432, C433, C434, C435, C436, C437, C438, C439, C440, C441, C442: symbol C-0402 -> pasv-cap:C-0402
- PCI0, PCI1, PCI2, PCI3: symbol CONN-5145154-1-PCI -> conn-te:CONN-5145154-1-PCI
- R401, R402, R403, R404: symbol R-0603 -> pasv-res:R-0603
- R405, R406, R407, R408, R409, R410, R411, R412, R413, R414, R415, R416, R417, R418, R419, R420, R421, R422, R423, R424, R425, R426, R427, R428, R429: symbol R-0402 -> pasv-res:R-0402
